Commit message: -Modified the PCA9685 package to take the i2c address from the .xacro and open the bus from there. -Added the on_configure and on_cleanup methods

File: src/hardware/urdf/ros2_control.xacro (robot description, xacro)
@@ -54,4 +54,68 @@
       <state_interface name="position"/>
     </joint>
+  </ros2_control>
+<ros2_control name="left_hand_mcp23017" type="system">
+    <hardware>
+      <plugin>pca9658_hardware_interface/PCA9685HardwareInterface</plugin>
+      <param name="i2c_address">32</param>  <!-- 0x20 in decimal -->
+    </hardware>
+    <joint name="left_hand_thumb_solenoid_joint">
+      <command_interface name="position"/>
+      <state_interface name="position"/>
+    </joint>
+    <joint name="left_hand_index_finger_solenoid_joint">
+      <command_interface name="position"/>
+      <state_interface name="position"/>
+    </joint>
+    <joint name="left_hand_middle_finger_solenoid_joint">
+      <command_interface name="position"/>
+      <state_interface name="position"/>
+    </joint>
+    <joint name="left_hand_ring_finger_solenoid_joint">
+      <command_interface name="position"/>
+      <state_interface name="position"/>
+    </joint>
+    <joint name="left_hand_pinky_solenoid_joint">
+      <command_interface name="position"/>
+      <state_interface name="position"/>
+    </joint>
+  </ros2_control>
+<ros2_control name="right_hand_mcp23017" type="system">
+    <hardware>
+      <plugin>pca9658_hardware_interface/PCA9685HardwareInterface</plugin>
+      <param name="i2c_address">33</param>  <!-- 0x21 in decimal -->
+    </hardware>
+    <joint name="right_hand_thumb_solenoid_joint">
+      <command_interface name="position"/>
+      <state_interface name="position"/>
+    </joint>
+    <joint name="right_hand_index_finger_solenoid_joint">
+      <command_interface name="position"/>
+      <state_interface name="position"/>
+    </joint>
+    <joint name="right_hand_middle_finger_solenoid_joint">
+      <command_interface name="position"/>
+      <state_interface name="position"/>
+    </joint>
+    <joint name="right_hand_ring_finger_solenoid_joint">
+      <command_interface name="position"/>
+      <state_interface name="position"/>
+    </joint>
+    <joint name="right_hand_pinky_solenoid_joint">
+      <command_interface name="position"/>
+      <state_interface name="position"/>
+    </joint>
+  </ros2_control>
+  <ros2_control name="left_hand_pca9685" type="system">
+    <hardware>
+      <plugin>pca9658_hardware_interface/PCA9685HardwareInterface</plugin>
+      <param name="i2c_bus">/dev/i2c-1</param>
+      <param name="i2c_address">64</param>  <!-- 0x40 in decimal -->
+      <param name="frequency_hz">50</param>
+      <!-- <param name="channels">
+        <channel name="joint_1" index="0" min_pulse="1000" max_pulse="2000" />
+        <channel name="joint_2" index="1" min_pulse="1000" max_pulse="2000" />
+      </param> -->
+    </hardware>
     <joint name="left_hand_thumb_servo_joint">
       <command_interface name="position"/>
@@ -74,4 +138,16 @@
       <state_interface name="position"/>
     </joint>
+  </ros2_control>
+  <ros2_control name="right_hand_pca9685" type="system">
+    <hardware>
+      <plugin>pca9658_hardware_interface/PCA9685HardwareInterface</plugin>
+      <param name="i2c_address">65</param>  <!-- 0x41 in decimal -->
+      <param name="frequency_hz">50</param>
+      <!-- we might want to define the parameters for these servos in this file
+      <param name="channels">
+        <channel name="joint_1" index="0" min_pulse="1000" max_pulse="2000" />
+        <channel name="joint_2" index="1" min_pulse="1000" max_pulse="2000" /> -->
+      <!-- </param> -->
+    </hardware>
     <joint name="right_hand_thumb_servo_joint">
       <command_interface name="position"/>

Commit message: -Fixed spelling errors and other mistakes

File: src/hardware/urdf/ros2_control.xacro (robot description, xacro)
@@ -55,59 +55,7 @@
     </joint>
   </ros2_control>
-<ros2_control name="left_hand_mcp23017" type="system">
-    <hardware>
-      <plugin>pca9658_hardware_interface/PCA9685HardwareInterface</plugin>
-      <param name="i2c_address">32</param>  <!-- 0x20 in decimal -->
-    </hardware>
-    <joint name="left_hand_thumb_solenoid_joint">
-      <command_interface name="position"/>
-      <state_interface name="position"/>
-    </joint>
-    <joint name="left_hand_index_finger_solenoid_joint">
-      <command_interface name="position"/>
-      <state_interface name="position"/>
-    </joint>
-    <joint name="left_hand_middle_finger_solenoid_joint">
-      <command_interface name="position"/>
-      <state_interface name="position"/>
-    </joint>
-    <joint name="left_hand_ring_finger_solenoid_joint">
-      <command_interface name="position"/>
-      <state_interface name="position"/>
-    </joint>
-    <joint name="left_hand_pinky_solenoid_joint">
-      <command_interface name="position"/>
-      <state_interface name="position"/>
-    </joint>
-  </ros2_control>
-<ros2_control name="right_hand_mcp23017" type="system">
-    <hardware>
-      <plugin>pca9658_hardware_interface/PCA9685HardwareInterface</plugin>
-      <param name="i2c_address">33</param>  <!-- 0x21 in decimal -->
-    </hardware>
-    <joint name="right_hand_thumb_solenoid_joint">
-      <command_interface name="position"/>
-      <state_interface name="position"/>
-    </joint>
-    <joint name="right_hand_index_finger_solenoid_joint">
-      <command_interface name="position"/>
-      <state_interface name="position"/>
-    </joint>
-    <joint name="right_hand_middle_finger_solenoid_joint">
-      <command_interface name="position"/>
-      <state_interface name="position"/>
-    </joint>
-    <joint name="right_hand_ring_finger_solenoid_joint">
-      <command_interface name="position"/>
-      <state_interface name="position"/>
-    </joint>
-    <joint name="right_hand_pinky_solenoid_joint">
-      <command_interface name="position"/>
-      <state_interface name="position"/>
-    </joint>
-  </ros2_control>
   <ros2_control name="left_hand_pca9685" type="system">
     <hardware>
-      <plugin>pca9658_hardware_interface/PCA9685HardwareInterface</plugin>
+      <plugin>pca9685_hardware_interface/Pca9685SystemHardware</plugin>
       <param name="i2c_bus">/dev/i2c-1</param>
       <param name="i2c_address">64</param>  <!-- 0x40 in decimal -->
@@ -119,27 +67,27 @@
     </hardware>
     <joint name="left_hand_thumb_servo_joint">
-      <command_interface name="position"/>
-      <state_interface name="position"/>
+      <command_interface name="velocity"/>
+      <state_interface name="velocity"/>
     </joint>
     <joint name="left_hand_index_finger_servo_joint">
-      <command_interface name="position"/>
-      <state_interface name="position"/>
+      <command_interface name="velocity"/>
+      <state_interface name="velocity"/>
     </joint>
     <joint name="left_hand_middle_finger_servo_joint">
-      <command_interface name="position"/>
-      <state_interface name="position"/>
+      <command_interface name="velocity"/>
+      <state_interface name="velocity"/>
     </joint>
     <joint name="left_hand_ring_finger_servo_joint">
-      <command_interface name="position"/>
-      <state_interface name="position"/>
+      <command_interface name="velocity"/>
+      <state_interface name="velocity"/>
     </joint>
     <joint name="left_hand_pinky_servo_joint">
-      <command_interface name="position"/>
-      <state_interface name="position"/>
+      <command_interface name="velocity"/>
+      <state_interface name="velocity"/>
     </joint>
   </ros2_control>
   <ros2_control name="right_hand_pca9685" type="system">
     <hardware>
-      <plugin>pca9658_hardware_interface/PCA9685HardwareInterface</plugin>
+      <plugin>pca9685_hardware_interface/Pca9685SystemHardware</plugin>
       <param name="i2c_address">65</param>  <!-- 0x41 in decimal -->
       <param name="frequency_hz">50</param>
@@ -151,22 +99,22 @@
     </hardware>
     <joint name="right_hand_thumb_servo_joint">
-      <command_interface name="position"/>
-      <state_interface name="position"/>
+      <command_interface name="velocity"/>
+      <state_interface name="velocity"/>
     </joint>
     <joint name="right_hand_index_finger_servo_joint">
-      <command_interface name="position"/>
-      <state_interface name="position"/>
+      <command_interface name="velocity"/>
+      <state_interface name="velocity"/>
     </joint>
     <joint name="right_hand_middle_finger_servo_joint">
-      <command_interface name="position"/>
-      <state_interface name="position"/>
+      <command_interface name="velocity"/>
+      <state_interface name="velocity"/>
     </joint>
     <joint name="right_hand_ring_finger_servo_joint">
-      <command_interface name="position"/>
-      <state_interface name="position"/>
+      <command_interface name="velocity"/>
+      <state_interface name="velocity"/>
     </joint>
     <joint name="right_hand_pinky_servo_joint">
-      <command_interface name="position"/>
-      <state_interface name="position"/>
+      <command_interface name="velocity"/>
+      <state_interface name="velocity"/>
     </joint>
   </ros2_control>
