Commit message: Fixed joint names

File: src/description/description/gazebo_control.xacro (robot description, xacro)
@@ -15,10 +15,10 @@
             <joint>left_hand_thumb_solenoid_joint</joint>
             <joint>left_hand_thumb_servo_joint</joint>
-            <joint>left_hand_index_solenoid_joint</joint>
-            <joint>left_hand_index_servo_joint</joint>
-            <joint>left_hand_middle_solenoid_joint</joint>
-            <joint>left_hand_middle_servo_joint</joint>
-            <joint>left_hand_ring_solenoid_joint</joint>
-            <joint>left_hand_ring_servo_joint</joint>
+            <joint>left_hand_index_finger_solenoid_joint</joint>
+            <joint>left_hand_index_finger_servo_joint</joint>
+            <joint>left_hand_middle_finger_solenoid_joint</joint>
+            <joint>left_hand_middle_finger_servo_joint</joint>
+            <joint>left_hand_ring_finger_solenoid_joint</joint>
+            <joint>left_hand_ring_finger_servo_joint</joint>
             <joint>left_hand_pinky_solenoid_joint</joint>
             <joint>left_hand_pinky_servo_joint</joint>
@@ -32,10 +32,10 @@
             <joint>right_hand_thumb_solenoid_joint</joint>
             <joint>right_hand_thumb_servo_joint</joint>
-            <joint>right_hand_index_solenoid_joint</joint>
-            <joint>right_hand_index_servo_joint</joint>
-            <joint>right_hand_middle_solenoid_joint</joint>
-            <joint>right_hand_middle_servo_joint</joint>
-            <joint>right_hand_ring_solenoid_joint</joint>
-            <joint>right_hand_ring_servo_joint</joint>
+            <joint>right_hand_index_finger_solenoid_joint</joint>
+            <joint>right_hand_index_finger_servo_joint</joint>
+            <joint>right_hand_middle_finger_solenoid_joint</joint>
+            <joint>right_hand_middle_finger_servo_joint</joint>
+            <joint>right_hand_ring_finger_solenoid_joint</joint>
+            <joint>right_hand_ring_finger_servo_joint</joint>
             <joint>right_hand_pinky_solenoid_joint</joint>
             <joint>right_hand_pinky_servo_joint</joint>

Commit message: Joints xacro refactorization

File: src/description/description/gazebo_control.xacro (robot description, xacro)
@@ -8,4 +8,12 @@
         </plugin>
     </gazebo>
+    <ros2_control name="GazeboSimSystem" type="system">
+        <hardware>
+            <plugin>gz_ros2_control/GazeboSimSystem</plugin>
+        </hardware>
+        <xacro:include filename="$(find hardware)/urdf/stepper_joints.xacro"/>
+        <xacro:include filename="$(find hardware)/urdf/solenoid_joints.xacro"/>
+        <xacro:include filename="$(find hardware)/urdf/servo_joints.xacro"/>
+    </ros2_control>
     <!-- Left Hand Controllers -->
     <gazebo>

File: src/hardware/urdf/ros2_control.xacro (robot description, xacro)
@@ -1,97 +1,11 @@
 <?xml version="1.0"?>
-<robot name="bothoven" xmlns:xacro="http://www.ros.org/wiki/xacro">
-  <xacro:include filename="$(find description)/urdf/bothoven.urdf.xacro"/>
+<robot xmlns:xacro="http://www.ros.org/wiki/xacro">
   <ros2_control name="hardware" type="system">
     <hardware>
         <plugin>hardware/BothovenHardware</plugin>
     </hardware>
-    <joint name="left_hand_stepper_joint">
-      <command_interface name="position"/>
-      <state_interface name="position"/>
-    </joint>
-    <joint name="right_hand_stepper_joint">
-      <command_interface name="position"/>
-      <state_interface name="position"/>
-    </joint>
-    <joint name="left_hand_thumb_solenoid_joint">
-      <command_interface name="position"/>
-      <state_interface name="position"/>
-    </joint>
-    <joint name="left_hand_index_finger_solenoid_joint">
-      <command_interface name="position"/>
-      <state_interface name="position"/>
-    </joint>
-    <joint name="left_hand_middle_finger_solenoid_joint">
-      <command_interface name="position"/>
-      <state_interface name="position"/>
-    </joint>
-    <joint name="left_hand_ring_finger_solenoid_joint">
-      <command_interface name="position"/>
-      <state_interface name="position"/>
-    </joint>
-    <joint name="left_hand_pinky_solenoid_joint">
-      <command_interface name="position"/>
-      <state_interface name="position"/>
-    </joint>
-    <joint name="right_hand_thumb_solenoid_joint">
-      <command_interface name="position"/>
-      <state_interface name="position"/>
-    </joint>
-    <joint name="right_hand_index_finger_solenoid_joint">
-      <command_interface name="position"/>
-      <state_interface name="position"/>
-    </joint>
-    <joint name="right_hand_middle_finger_solenoid_joint">
-      <command_interface name="position"/>
-      <state_interface name="position"/>
-    </joint>
-    <joint name="right_hand_ring_finger_solenoid_joint">
-      <command_interface name="position"/>
-      <state_interface name="position"/>
-    </joint>
-    <joint name="right_hand_pinky_solenoid_joint">
-      <command_interface name="position"/>
-      <state_interface name="position"/>
-    </joint>
-    <joint name="left_hand_thumb_servo_joint">
-      <command_interface name="position"/>
-      <state_interface name="position"/>
-    </joint>
-    <joint name="left_hand_index_finger_servo_joint">
-      <command_interface name="position"/>
-      <state_interface name="position"/>
-    </joint>
-    <joint name="left_hand_middle_finger_servo_joint">
-      <command_interface name="position"/>
-      <state_interface name="position"/>
-    </joint>
-    <joint name="left_hand_ring_finger_servo_joint">
-      <command_interface name="position"/>
-      <state_interface name="position"/>
-    </joint>
-    <joint name="left_hand_pinky_servo_joint">
-      <command_interface name="position"/>
-      <state_interface name="position"/>
-    </joint>
-    <joint name="right_hand_thumb_servo_joint">
-      <command_interface name="position"/>
-      <state_interface name="position"/>
-    </joint>
-    <joint name="right_hand_index_finger_servo_joint">
-      <command_interface name="position"/>
-      <state_interface name="position"/>
-    </joint>
-    <joint name="right_hand_middle_finger_servo_joint">
-      <command_interface name="position"/>
-      <state_interface name="position"/>
-    </joint>
-    <joint name="right_hand_ring_finger_servo_joint">
-      <command_interface name="position"/>
-      <state_interface name="position"/>
-    </joint>
-    <joint name="right_hand_pinky_servo_joint">
-      <command_interface name="position"/>
-      <state_interface name="position"/>
-    </joint>
+    <xacro:include filename="$(find hardware)/urdf/stepper_joints.xacro"/>
+    <xacro:include filename="$(find hardware)/urdf/solenoid_joints.xacro"/>
+    <xacro:include filename="$(find hardware)/urdf/servo_joints.xacro"/>
   </ros2_control>
 </robot>

Commit message: Fixed the physics engine and ros2_control in GZ

File: src/description/description/gazebo_control.xacro (robot description, xacro)
@@ -1,13 +1,4 @@
 <?xml version="1.0"?>
 <robot xmlns:xacro="http://www.ros.org/wiki/xacro">
-    <gazebo>
-        <plugin name="gz_ros2_control::GazeboSimROS2ControlPlugin" filename="libgz_ros2_control-system.so">
-            <parameters>$(find hardware)/config/controllers.yaml</parameters>
-            <ros>
-                <namespace>bothoven</namespace>
-                <remapping>/robot_description:=/robot_description</remapping>
-            </ros>
-        </plugin>
-    </gazebo>
     <ros2_control name="GazeboSimSystem" type="system">
         <hardware>
@@ -18,37 +9,8 @@
         <xacro:include filename="$(find hardware)/urdf/servo_joints.xacro"/>
     </ros2_control>
-    <!-- Left Hand Controllers -->
-    <!-- <gazebo>
-        <plugin name="left_hand_controller" filename="libgazebo_ros_joint_trajectory_controller.so">
-            <robotNamespace>/left_hand</robotNamespace>
-            <joint>left_hand_stepper_joint</joint>
-            <joint>left_hand_thumb_solenoid_joint</joint>
-            <joint>left_hand_thumb_servo_joint</joint>
-            <joint>left_hand_index_finger_solenoid_joint</joint>
-            <joint>left_hand_index_finger_servo_joint</joint>
-            <joint>left_hand_middle_finger_solenoid_joint</joint>
-            <joint>left_hand_middle_finger_servo_joint</joint>
-            <joint>left_hand_ring_finger_solenoid_joint</joint>
-            <joint>left_hand_ring_finger_servo_joint</joint>
-            <joint>left_hand_pinky_solenoid_joint</joint>
-            <joint>left_hand_pinky_servo_joint</joint>
+    <gazebo>
+        <plugin name="gz_ros2_control::GazeboSimROS2ControlPlugin" filename="gz_ros2_control-system">
+            <parameters>$(find hardware)/config/controllers.yaml</parameters>
         </plugin>
-    </gazebo> -->
-    <!-- Right Hand Controllers -->
-    <!-- <gazebo>
-        <plugin name="right_hand_controller" filename="libgazebo_ros_joint_trajectory_controller.so">
-            <robotNamespace>/right_hand</robotNamespace>
-            <joint>right_hand_stepper_joint</joint>
-            <joint>right_hand_thumb_solenoid_joint</joint>
-            <joint>right_hand_thumb_servo_joint</joint>
-            <joint>right_hand_index_finger_solenoid_joint</joint>
-            <joint>right_hand_index_finger_servo_joint</joint>
-            <joint>right_hand_middle_finger_solenoid_joint</joint>
-            <joint>right_hand_middle_finger_servo_joint</joint>
-            <joint>right_hand_ring_finger_solenoid_joint</joint>
-            <joint>right_hand_ring_finger_servo_joint</joint>
-            <joint>right_hand_pinky_solenoid_joint</joint>
-            <joint>right_hand_pinky_servo_joint</joint>
-        </plugin>
-    </gazebo> -->
+    </gazebo>
 </robot>
