Commit message: Added collisions to hands and fingers

File: src/description/description/common.xacro (robot description, xacro)
@@ -70,4 +70,9 @@
                     <material name="blue"/>
                 </visual>
+                <collision>
+                    <geometry>
+                        <box size="0.1 0.05 0.05"/>
+                    </geometry>
+                </collision>
             </link>
             <joint name="${name}_joint" type="prismatic">
@@ -89,4 +94,10 @@
                     <material name="orange"/>
                 </visual>
+                <collision>
+                    <geometry>
+                        <box size="${hand_length} ${hand_width} ${hand_height}"/>
+                    </geometry>
+                    <origin xyz="0 0.5 0"/>
+                </collision>
             </link>
             <joint name="${name}_joint" type="fixed">
@@ -141,4 +152,10 @@
                     <material name="black"/>
                 </visual>
+                <collision>
+                    <geometry>
+                        <box size="${finger_thickness} ${finger_length} ${finger_thickness}"/>
+                    </geometry>
+                    <origin xyz="0 -0.05 0"/>
+                </collision>
             </link>
             <joint name="${name}_joint" type="fixed">

Commit message: Added intertia to fingers, hands, and carriages

File: src/description/description/common.xacro (robot description, xacro)
@@ -75,4 +75,9 @@
                     </geometry>
                 </collision>
+                <inertial>
+                    <mass value="0.5"/>
+                    <origin xyz="0 0 0"/>
+                    <inertia ixx="0.001" ixy="0.0" ixz="0.0" iyy="0.001" iyz="0.0" izz="0.001"/>
+                </inertial>
             </link>
             <joint name="${name}_joint" type="prismatic">
@@ -100,4 +105,9 @@
                     <origin xyz="0 0.5 0"/>
                 </collision>
+                <inertial>
+                    <mass value="0.2"/>
+                    <origin xyz="0 0 0"/>
+                    <inertia ixx="0.0005" ixy="0.0" ixz="0.0" iyy="0.0005" iyz="0.0" izz="0.0005"/>
+                </inertial>
             </link>
             <joint name="${name}_joint" type="fixed">
@@ -158,4 +168,9 @@
                     <origin xyz="0 -0.05 0"/>
                 </collision>
+                <inertial>
+                    <mass value="0.1"/>
+                    <origin xyz="0 0 0"/>
+                    <inertia ixx="0.0001" ixy="0.0" ixz="0.0" iyy="0.0001" iyz="0.0" izz="0.0001"/>
+                </inertial>
             </link>
             <joint name="${name}_joint" type="fixed">

Commit message: Added min/max values to actuated joints

File: src/description/description/common.xacro (robot description, xacro)
@@ -42,4 +42,10 @@
         <xacro:property name="ring_offset" value="${hand_length/2 - 2*finger_spacing}"/>
         <xacro:property name="pinky_offset" value="${hand_length/2 - finger_spacing}"/>
+    <!-- Servo Joint Properties -->
+        <xacro:property name="servo_min" value="-0.2"/>
+        <xacro:property name="servo_max" value="0.2"/>
+    <!-- Solenoid Joint Properties -->
+        <xacro:property name="solenoid_min" value="-0.2"/>
+        <xacro:property name="solenoid_max" value="0.2"/>
   <!-- Macros -->
     <!-- Stepper Motor Macro -->
@@ -154,5 +160,5 @@
                 <origin xyz="0 0 0"/>
                 <axis xyz="1 0 0"/>
-                <limit lower="-0.2" upper="0.2" effort="1" velocity="1.0"/>
+                <limit lower="${solenoid_min}" upper="${solenoid_max}" effort="1" velocity="1.0"/>
             </joint>
         </xacro:macro>
@@ -180,5 +186,5 @@
                 <origin xyz="${x_origin} -${hand_width/2} -0.01"/>
                 <axis xyz="0 0 1"/>
-                <limit lower="-0.2" upper="0.2" effort="1" velocity="1.0"/>
+                <limit lower="${servo_min}" upper="${servo_max}" effort="1" velocity="1.0"/>
             </joint>
         </xacro:macro>

File: src/hardware/urdf/servo_joints.xacro (robot description, xacro)
@@ -2,41 +2,71 @@
 <robot xmlns:xacro="http://www.ros.org/wiki/xacro">
     <joint name="left_hand_thumb_servo_joint">
-        <command_interface name="position"/>
+        <command_interface name="position">
+            <param name="min">${servo_min}</param>
+            <param name="max">${servo_max}</param>
+        </command_interface>
         <state_interface name="position"/>
     </joint>
     <joint name="left_hand_index_finger_servo_joint">
-        <command_interface name="position"/>
+        <command_interface name="position">
+            <param name="min">${servo_min}</param>
+            <param name="max">${servo_max}</param>
+        </command_interface>
         <state_interface name="position"/>
     </joint>
     <joint name="left_hand_middle_finger_servo_joint">
-        <command_interface name="position"/>
+        <command_interface name="position">
+            <param name="min">${servo_min}</param>
+            <param name="max">${servo_max}</param>
+        </command_interface>
         <state_interface name="position"/>
     </joint>
     <joint name="left_hand_ring_finger_servo_joint">
-        <command_interface name="position"/>
+        <command_interface name="position">
+            <param name="min">${servo_min}</param>
+            <param name="max">${servo_max}</param>
+        </command_interface>
         <state_interface name="position"/>
     </joint>
     <joint name="left_hand_pinky_servo_joint">
-        <command_interface name="position"/>
+        <command_interface name="position">
+            <param name="min">${servo_min}</param>
+            <param name="max">${servo_max}</param>
+        </command_interface>
         <state_interface name="position"/>
     </joint>
     <joint name="right_hand_thumb_servo_joint">
-        <command_interface name="position"/>
+        <command_interface name="position">
+            <param name="min">${servo_min}</param>
+            <param name="max">${servo_max}</param>
+        </command_interface>
         <state_interface name="position"/>
     </joint>
     <joint name="right_hand_index_finger_servo_joint">
-        <command_interface name="position"/>
+        <command_interface name="position">
+            <param name="min">${servo_min}</param>
+            <param name="max">${servo_max}</param>
+        </command_interface>
         <state_interface name="position"/>
     </joint>
     <joint name="right_hand_middle_finger_servo_joint">
-        <command_interface name="position"/>
+        <command_interface name="position">
+            <param name="min">${servo_min}</param>
+            <param name="max">${servo_max}</param>
+        </command_interface>
         <state_interface name="position"/>
     </joint>
     <joint name="right_hand_ring_finger_servo_joint">
-        <command_interface name="position"/>
+        <command_interface name="position">
+            <param name="min">${servo_min}</param>
+            <param name="max">${servo_max}</param>
+        </command_interface>
         <state_interface name="position"/>
     </joint>
     <joint name="right_hand_pinky_servo_joint">
-        <command_interface name="position"/>
+        <command_interface name="position">
+            <param name="min">${servo_min}</param>
+            <param name="max">${servo_max}</param>
+        </command_interface>
         <state_interface name="position"/>
     </joint>

File: src/hardware/urdf/solenoid_joints.xacro (robot description, xacro)
@@ -2,41 +2,71 @@
 <robot xmlns:xacro="http://www.ros.org/wiki/xacro">
     <joint name="left_hand_thumb_solenoid_joint">
-        <command_interface name="position"/>
+        <command_interface name="position">
+            <param name="min">${solenoid_min}</param>
+            <param name="max">${solenoid_max}</param>
+        </command_interface>
         <state_interface name="position"/>
     </joint>
     <joint name="left_hand_index_finger_solenoid_joint">
-        <command_interface name="position"/>
+        <command_interface name="position">
+            <param name="min">${solenoid_min}</param>
+            <param name="max">${solenoid_max}</param>
+        </command_interface>
         <state_interface name="position"/>
     </joint>
     <joint name="left_hand_middle_finger_solenoid_joint">
-        <command_interface name="position"/>
+        <command_interface name="position">
+            <param name="min">${solenoid_min}</param>
+            <param name="max">${solenoid_max}</param>
+        </command_interface>
         <state_interface name="position"/>
     </joint>
     <joint name="left_hand_ring_finger_solenoid_joint">
-        <command_interface name="position"/>
+        <command_interface name="position">
+            <param name="min">${solenoid_min}</param>
+            <param name="max">${solenoid_max}</param>
+        </command_interface>
         <state_interface name="position"/>
     </joint>
     <joint name="left_hand_pinky_solenoid_joint">
-        <command_interface name="position"/>
+        <command_interface name="position">
+            <param name="min">${solenoid_min}</param>
+            <param name="max">${solenoid_max}</param>
+        </command_interface>
         <state_interface name="position"/>
     </joint>
     <joint name="right_hand_thumb_solenoid_joint">
-        <command_interface name="position"/>
+        <command_interface name="position">
+            <param name="min">${solenoid_min}</param>
+            <param name="max">${solenoid_max}</param>
+        </command_interface>
         <state_interface name="position"/>
     </joint>
     <joint name="right_hand_index_finger_solenoid_joint">
-        <command_interface name="position"/>
+        <command_interface name="position">
+            <param name="min">${solenoid_min}</param>
+            <param name="max">${solenoid_max}</param>
+        </command_interface>
         <state_interface name="position"/>
     </joint>
     <joint name="right_hand_middle_finger_solenoid_joint">
-        <command_interface name="position"/>
+        <command_interface name="position">
+            <param name="min">${solenoid_min}</param>
+            <param name="max">${solenoid_max}</param>
+        </command_interface>
         <state_interface name="position"/>
     </joint>
     <joint name="right_hand_ring_finger_solenoid_joint">
-        <command_interface name="position"/>
+        <command_interface name="position">
+            <param name="min">${solenoid_min}</param>
+            <param name="max">${solenoid_max}</param>
+        </command_interface>
         <state_interface name="position"/>
     </joint>
     <joint name="right_hand_pinky_solenoid_joint">
-        <command_interface name="position"/>
+        <command_interface name="position">
+            <param name="min">${solenoid_min}</param>
+            <param name="max">${solenoid_max}</param>
+        </command_interface>
         <state_interface name="position"/>
     </joint>

File: src/hardware/urdf/stepper_joints.xacro (robot description, xacro)
@@ -2,9 +2,15 @@
 <robot xmlns:xacro="http://www.ros.org/wiki/xacro">
     <joint name="left_hand_stepper_joint">
-        <command_interface name="position"/>
+        <command_interface name="position">
+            <param name="min">${stepper_min_angle}</param>
+            <param name="max">${stepper_max_angle}</param>
+        </command_interface>
         <state_interface name="position"/>
     </joint>
     <joint name="right_hand_stepper_joint">
-        <command_interface name="position"/>
+        <command_interface name="position">
+            <param name="min">${stepper_min_angle}</param>
+            <param name="max">${stepper_max_angle}</param>
+        </command_interface>
         <state_interface name="position"/>
     </joint>
