Commit message: Refactored Core description

File: src/description/description/bothoven_core.xacro (robot description, xacro)
@@ -1,24 +1,6 @@
 <?xml version="1.0"?>
 <robot xmlns:xacro="http://www.ros.org/wiki/xacro">
-  <!-- Colours -->
-  <material name="white">
-    <color rgba="1 1 1 1"/>
-  </material>
-  <material name="orange">
-      <color rgba="1 0.3 0.1 1"/>
-  </material>
-  <material name="blue">
-      <color rgba="0.2 0.2 1 1"/>
-  </material>
-  <material name="black">
-      <color rgba="0 0 0 1"/>
-  </material>
-  <material name="yellow">
-    <color rgba="1.0 1.0 0.0 1.0"/>
-  </material>
-  <material name="green">
-    <color rgba="0.0 1.0 0.0 1.0"/>
-  </material>
- <!-- Robot Properties -->
+  <xacro:include filename="$(find description)/description/common.xacro"/>
+  <!-- Robot Properties -->
   <link name="base_link"/>
   <!-- Aluminum Rail -->
@@ -37,153 +19,13 @@
   </joint>
   <!-- Stepper Motors -->
-  <xacro:property name="stepper_min_angle" value="0"/>
-  <xacro:property name="stepper_max_angle" value="6.28"/>
-  <xacro:macro name="stepper" params="name parent_link origin_xyz">
-    <link name="${name}">
-      <visual>
-        <geometry>
-          <cylinder radius="0.02" length="0.05"/>
-        </geometry>
-        <material name="black"/>
-      </visual>
-    </link>
-    <joint name="${name}_joint" type="revolute">
-      <parent link="${parent_link}"/>
-      <child link="${name}"/>
-      <origin xyz="${origin_xyz}" rpy="0 0 0"/>
-      <axis xyz="0 0 1"/>
-      <limit lower="${stepper_min_angle}" upper="${stepper_max_angle}" effort="5" velocity="1.0"/>
-    </joint>
-  </xacro:macro>
   <xacro:stepper name="left_hand_stepper" parent_link="aluminum_rail" origin_xyz="0.75 0 0"/>
   <xacro:stepper name="right_hand_stepper" parent_link="aluminum_rail" origin_xyz="-0.75 0 0"/>
   <!-- Carriages -->
-  <xacro:property name="carriage_min_position" value="-0.68"/>
-  <xacro:property name="carriage_max_position" value="0.68"/>
-  <xacro:property name="carriage_stepper_offset" value="${carriage_max_position}"/> <!-- Assuming a min angle of 0 rad for the stepper -->
-  <xacro:property name="carriage_stepper_multiplier" value="${(carriage_min_position - carriage_stepper_offset) / stepper_max_angle}"/>
-  <link name="left_carriage">
-    <visual>
-      <geometry>
-        <box size="0.1 0.05 0.05"/>
-      </geometry>
-      <material name="blue"/>
-    </visual>
-  </link>
-  <link name="right_carriage">
-    <visual>
-      <geometry>
-        <box size="0.1 0.05 0.05"/>
-      </geometry>
-      <material name="blue"/>
-    </visual>
-  </link>
-  <joint name="left_carriage_joint" type="prismatic">
-    <parent link="aluminum_rail"/>
-    <child link="left_carriage"/>
-    <origin xyz="0 0 0"/>
-    <axis xyz="1 0 0"/>
-    <limit lower="${carriage_min_position}" upper="${carriage_max_position}" effort="10" velocity="0.5"/>
-    <mimic joint="left_hand_stepper_joint" multiplier="${carriage_stepper_multiplier}" offset="${carriage_stepper_offset}"/>
-  </joint>
-  <joint name="right_carriage_joint" type="prismatic">
-    <parent link="aluminum_rail"/>
-    <child link="right_carriage"/>
-    <origin xyz="0 0 0"/>
-    <axis xyz="-1 0 0"/>
-    <limit lower="${carriage_min_position}" upper="${carriage_max_position}" effort="10" velocity="0.5"/>
-    <mimic joint="right_hand_stepper_joint" multiplier="${carriage_stepper_multiplier}" offset="${carriage_stepper_offset}"/>
-  </joint>
+  <xacro:carriage name="left_carriage" parent_link="aluminum_rail" axis_x="1" mimic="left_hand_stepper_joint"/>
+  <xacro:carriage name="right_carriage" parent_link="aluminum_rail" axis_x="-1" mimic="right_hand_stepper_joint"/>
   <!-- Hands -->
-  <xacro:property name="hand_length" value="0.2"/>
-  <xacro:property name="hand_width" value="0.1"/>
-  <xacro:property name="hand_height" value="0.05"/>
-  <link name="left_hand">
-    <visual>
-      <geometry>
-        <box size="${hand_length} ${hand_width} ${hand_height}"/>
-      </geometry>
-      <material name="orange"/>
-    </visual>
-  </link>
-  <link name="right_hand">
-    <visual>
-      <geometry>
-        <box size="${hand_length} ${hand_width} ${hand_height}"/>
-      </geometry>
-      <material name="orange"/>
-    </visual>
-  </link>
-  <joint name="left_hand_joint" type="fixed">
-    <parent link="left_carriage"/>
-    <child link="left_hand"/>
-    <origin xyz="0 0.5 0"/>
-  </joint>
-  <joint name="right_hand_joint" type="fixed">
-    <parent link="right_carriage"/>
-    <child link="right_hand"/>
-    <origin xyz="0 0.5 0"/>
-  </joint>
-  <!-- Solenoids for Finger Press -->
-  <xacro:macro name="solenoid" params="name parent_link">
-    <link name="${name}">
-      <visual>
-        <geometry>
-          <cylinder radius="0.01" length="0.025"/>
-        </geometry>
-        <material name="green"/>
-      </visual>
-    </link>
-    <joint name="${name}_joint" type="revolute">
-      <parent link="${parent_link}"/>
-      <child link="${name}"/>
-      <origin xyz="0 0 0"/>
-      <axis xyz="1 0 0"/>
-      <limit lower="-0.2" upper="0.2" effort="1" velocity="1.0"/>
-    </joint>
-  </xacro:macro>
-  <!-- Servos for Lateral Motion -->
-  <xacro:macro name="servo" params="name parent_link x_origin">
-    <link name="${name}">
-      <visual>
-        <geometry>
-          <box size="0.02 0.02 0.02"/>
-        </geometry>
-        <material name="yellow"/>
-      </visual>
-    </link>
-    <joint name="${name}_joint" type="revolute">
-      <parent link="${parent_link}"/>
-      <child link="${name}"/>
-      <origin xyz="${x_origin} -${hand_width/2} -0.01"/>
-      <axis xyz="0 0 1"/>
-      <limit lower="-0.2" upper="0.2" effort="1" velocity="1.0"/>
-    </joint>
-  </xacro:macro>
-  <!-- Fingers -->
-  <xacro:property name="finger_length" value="0.1"/>
-  <xacro:property name="finger_thickness" value="0.01"/>
-  <xacro:macro name="finger" params="name parent_link">
-    <link name="${name}">
-      <visual>
-        <geometry>
-          <box size="${finger_thickness} ${finger_length} ${finger_thickness}"/>
-        </geometry>
-        <material name="black"/>
-      </visual>
-    </link>
-    <joint name="${name}_joint" type="fixed">
-      <parent link="${parent_link}"/>
-      <child link="${name}"/>
-      <origin xyz="0 -0.05 0"/>
-    </joint>
-  </xacro:macro>
-  <!-- Solenoids and Servos attached to each finger for key press and lateral motion -->
-  <xacro:property name="finger_spacing" value="${hand_length/6}"/>
-  <xacro:property name="thumb_offset" value="${-hand_length/2 + finger_spacing}"/>
-  <xacro:property name="index_offset" value="${-hand_length/2 + 2*finger_spacing}"/>
-  <xacro:property name="middle_offset" value="0"/>
-  <xacro:property name="ring_offset" value="${hand_length/2 - 2*finger_spacing}"/>
-  <xacro:property name="pinky_offset" value="${hand_length/2 - finger_spacing}"/>
+  <xacro:hand name="left_hand" parent_link="left_carriage"/>
+  <xacro:hand name="right_hand" parent_link="right_carriage"/>
+  <!-- Solenoids and Servos attached to each finger -->
   <xacro:solenoid name="left_hand_thumb_solenoid" parent_link="left_hand_thumb_servo"/>
   <xacro:servo name="left_hand_thumb_servo" parent_link="left_hand" x_origin="${thumb_offset}"/>

Commit message: Added Gazebo support (WIP)

File: src/description/description/bothoven_core.xacro (robot description, xacro)
@@ -3,5 +3,11 @@
   <xacro:include filename="$(find description)/description/common.xacro"/>
   <!-- Robot Properties -->
-  <link name="base_link"/>
+  <link name="base_link">
+    <inertial>
+      <mass value="1.0"/>
+      <origin xyz="0 0 0"/>
+      <inertia ixx="0.1" ixy="0.0" ixz="0.0" iyy="0.1" iyz="0.0" izz="0.1"/>
+    </inertial>
+  </link>
   <!-- Aluminum Rail -->
   <link name="aluminum_rail">
@@ -12,4 +18,7 @@
       <material name="white"/>
     </visual>
+    <gazebo>
+      <material>Gazebo/White</material>
+    </gazebo>
   </link>
   <joint name="rail_to_base" type="fixed">
@@ -17,4 +26,7 @@
     <child link="aluminum_rail"/>
     <origin xyz="0 0 0.1"/>
+    <gazebo>
+      <disableFixedJointLumping>false</disableFixedJointLumping>
+    </gazebo>
   </joint>
   <!-- Stepper Motors -->

File: src/description/description/common.xacro (robot description, xacro)
@@ -52,4 +52,12 @@
                     <material name="black"/>
                 </visual>
+                <inertial>
+                    <mass value="0.1"/>
+                    <origin xyz="0 0 0"/>
+                    <inertia ixx="0.0001" ixy="0.0" ixz="0.0" iyy="0.0001" iyz="0.0" izz="0.0001"/>
+                </inertial>
+                <gazebo>
+                    <material>Gazebo/Black</material>
+                </gazebo>
             </link>
             <joint name="${name}_joint" type="revolute">
@@ -80,4 +88,7 @@
                     <inertia ixx="0.001" ixy="0.0" ixz="0.0" iyy="0.001" iyz="0.0" izz="0.001"/>
                 </inertial>
+                <gazebo>
+                    <material>Gazebo/Blue</material>
+                </gazebo>
             </link>
             <joint name="${name}_joint" type="prismatic">
@@ -110,4 +121,7 @@
                     <inertia ixx="0.0005" ixy="0.0" ixz="0.0" iyy="0.0005" iyz="0.0" izz="0.0005"/>
                 </inertial>
+                <gazebo>
+                    <material>Gazebo/Orange</material>
+                </gazebo>
             </link>
             <joint name="${name}_joint" type="fixed">
@@ -126,4 +140,12 @@
                     <material name="green"/>
                 </visual>
+                <inertial>
+                    <mass value="0.05"/>
+                    <origin xyz="0 0 0"/>
+                    <inertia ixx="0.00005" ixy="0.0" ixz="0.0" iyy="0.00005" iyz="0.0" izz="0.00005"/>
+                </inertial>
+                <gazebo>
+                    <material>Gazebo/Green</material>
+                </gazebo>
             </link>
             <joint name="${name}_joint" type="revolute">
@@ -144,4 +166,12 @@
                     <material name="yellow"/>
                 </visual>
+                <inertial>
+                    <mass value="0.05"/>
+                    <origin xyz="0 0 0"/>
+                    <inertia ixx="0.00002" ixy="0.0" ixz="0.0" iyy="0.00002" iyz="0.0" izz="0.00002"/>
+                </inertial>
+                <gazebo>
+                    <material>Gazebo/Yellow</material>
+                </gazebo>
             </link>
             <joint name="${name}_joint" type="revolute">
@@ -173,4 +203,7 @@
                     <inertia ixx="0.0001" ixy="0.0" ixz="0.0" iyy="0.0001" iyz="0.0" izz="0.0001"/>
                 </inertial>
+                <gazebo>
+                    <material>Gazebo/Black</material>
+                </gazebo>
             </link>
             <joint name="${name}_joint" type="fixed">

File: src/description/description/gazebo_control.xacro (robot description, xacro)
@@ -3,7 +3,9 @@
     <gazebo>
         <plugin name="gz_ros2_control::GazeboSimROS2ControlPlugin" filename="libgz_ros2_control-system.so">
-            <robotNamespace>/</robotNamespace>
-            <parameters></parameters>
-            <controller_manager_prefix_node_name>controller_manager</controller_manager_prefix_node_name>
+            <parameters>$(find hardware)/config/controllers.yaml</parameters>
+            <ros>
+                <namespace>bothoven</namespace>
+                <remapping>/robot_description:=/robot_description</remapping>
+            </ros>
         </plugin>
     </gazebo>
@@ -17,5 +19,5 @@
     </ros2_control>
     <!-- Left Hand Controllers -->
-    <gazebo>
+    <!-- <gazebo>
         <plugin name="left_hand_controller" filename="libgazebo_ros_joint_trajectory_controller.so">
             <robotNamespace>/left_hand</robotNamespace>
@@ -32,7 +34,7 @@
             <joint>left_hand_pinky_servo_joint</joint>
         </plugin>
-    </gazebo>
+    </gazebo> -->
     <!-- Right Hand Controllers -->
-    <gazebo>
+    <!-- <gazebo>
         <plugin name="right_hand_controller" filename="libgazebo_ros_joint_trajectory_controller.so">
             <robotNamespace>/right_hand</robotNamespace>
@@ -49,4 +51,4 @@
             <joint>right_hand_pinky_servo_joint</joint>
         </plugin>
-    </gazebo>
+    </gazebo> -->
 </robot>

File: src/description/urdf/bothoven.urdf.xacro (robot description, xacro)
@@ -1,5 +1,12 @@
 <?xml version="1.0"?>
 <robot name="bothoven" xmlns:xacro="http://www.ros.org/wiki/xacro">
+  <xacro:arg name="use_ros2_control" default="true"/>
+  <xacro:arg name="sim_mode" default="false"/>
   <xacro:include filename="$(find description)/description/bothoven_core.xacro"/>
-  <!-- <xacro:include filename="$(find description)/description/gazebo_control.xacro"/> -->
+  <xacro:if value="$(arg use_ros2_control)">
+      <xacro:include filename="$(find hardware)/urdf/ros2_control.xacro"/>
+  </xacro:if>
+  <xacro:unless value="$(arg use_ros2_control)">
+      <xacro:include filename="$(find description)/description/gazebo_control.xacro" />
+  </xacro:unless>
 </robot>

Commit message: formatted file and Inverted each carriage x axis

File: src/description/description/bothoven_core.xacro (robot description, xacro)
@@ -1,11 +1,11 @@
 <?xml version="1.0"?>
 <robot xmlns:xacro="http://www.ros.org/wiki/xacro">
-  <xacro:include filename="$(find description)/description/common.xacro"/>
+  <xacro:include filename="$(find description)/description/common.xacro" />
   <!-- Robot Properties -->
   <link name="base_link">
     <inertial>
-      <mass value="1.0"/>
-      <origin xyz="0 0 0"/>
-      <inertia ixx="0.1" ixy="0.0" ixz="0.0" iyy="0.1" iyz="0.0" izz="0.1"/>
+      <mass value="1.0" />
+      <origin xyz="0 0 0" />
+      <inertia ixx="0.1" ixy="0.0" ixz="0.0" iyy="0.1" iyz="0.0" izz="0.1" />
     </inertial>
   </link>
@@ -14,7 +14,7 @@
     <visual>
       <geometry>
-        <box size="1.5 0.02 0.02"/>
+        <box size="1.5 0.02 0.02" />
       </geometry>
-      <material name="white"/>
+      <material name="white" />
     </visual>
     <gazebo>
@@ -23,7 +23,7 @@
   </link>
   <joint name="rail_to_base" type="fixed">
-    <parent link="base_link"/>
-    <child link="aluminum_rail"/>
-    <origin xyz="0 0 0.1"/>
+    <parent link="base_link" />
+    <child link="aluminum_rail" />
+    <origin xyz="0 0 0.1" />
     <gazebo>
       <disableFixedJointLumping>false</disableFixedJointLumping>
@@ -31,44 +31,54 @@
   </joint>
   <!-- Stepper Motors -->
-  <xacro:stepper name="left_hand_stepper" parent_link="aluminum_rail" origin_xyz="0.75 0 0"/>
-  <xacro:stepper name="right_hand_stepper" parent_link="aluminum_rail" origin_xyz="-0.75 0 0"/>
+  <xacro:stepper name="left_hand_stepper" parent_link="aluminum_rail" origin_xyz="0.75 0 0" />
+  <xacro:stepper name="right_hand_stepper" parent_link="aluminum_rail" origin_xyz="-0.75 0 0" />
   <!-- Carriages -->
-  <xacro:carriage name="left_carriage" parent_link="aluminum_rail" axis_x="1" mimic="left_hand_stepper_joint"/>
-  <xacro:carriage name="right_carriage" parent_link="aluminum_rail" axis_x="-1" mimic="right_hand_stepper_joint"/>
+  <xacro:carriage name="left_carriage" parent_link="aluminum_rail" axis_x="-1"
+    mimic="left_hand_stepper_joint" />
+  <xacro:carriage name="right_carriage" parent_link="aluminum_rail" axis_x="1"
+    mimic="right_hand_stepper_joint" />
   <!-- Hands -->
-  <xacro:hand name="left_hand" parent_link="left_carriage"/>
-  <xacro:hand name="right_hand" parent_link="right_carriage"/>
+  <xacro:hand name="left_hand" parent_link="left_carriage" />
+  <xacro:hand name="right_hand" parent_link="right_carriage" />
   <!-- Solenoids and Servos attached to each finger -->
-  <xacro:solenoid name="left_hand_thumb_solenoid" parent_link="left_hand_thumb_servo"/>
-  <xacro:servo name="left_hand_thumb_servo" parent_link="left_hand" x_origin="${thumb_offset}"/>
-  <xacro:solenoid name="left_hand_index_finger_solenoid" parent_link="left_hand_index_finger_servo"/>
-  <xacro:servo name="left_hand_index_finger_servo" parent_link="left_hand" x_origin="${index_offset}"/>
-  <xacro:solenoid name="left_hand_middle_finger_solenoid" parent_link="left_hand_middle_finger_servo"/>
-  <xacro:servo name="left_hand_middle_finger_servo" parent_link="left_hand" x_origin="${middle_offset}"/>
-  <xacro:solenoid name="left_hand_ring_finger_solenoid" parent_link="left_hand_ring_finger_servo"/>
-  <xacro:servo name="left_hand_ring_finger_servo" parent_link="left_hand" x_origin="${ring_offset}"/>
-  <xacro:solenoid name="left_hand_pinky_solenoid" parent_link="left_hand_pinky_servo"/>
-  <xacro:servo name="left_hand_pinky_servo" parent_link="left_hand" x_origin="${pinky_offset}"/>
-  <xacro:solenoid name="right_hand_thumb_solenoid" parent_link="right_hand_thumb_servo"/>
-  <xacro:servo name="right_hand_thumb_servo" parent_link="right_hand" x_origin="${-thumb_offset}"/>
-  <xacro:solenoid name="right_hand_index_finger_solenoid" parent_link="right_hand_index_finger_servo"/>
-  <xacro:servo name="right_hand_index_finger_servo" parent_link="right_hand" x_origin="${-index_offset}"/>
-  <xacro:solenoid name="right_hand_middle_finger_solenoid" parent_link="right_hand_middle_finger_servo"/>
-  <xacro:servo name="right_hand_middle_finger_servo" parent_link="right_hand" x_origin="${-middle_offset}"/>
-  <xacro:solenoid name="right_hand_ring_finger_solenoid" parent_link="right_hand_ring_finger_servo"/>
-  <xacro:servo name="right_hand_ring_finger_servo" parent_link="right_hand" x_origin="${-ring_offset}"/>
-  <xacro:solenoid name="right_hand_pinky_solenoid" parent_link="right_hand_pinky_servo"/>
-  <xacro:servo name="right_hand_pinky_servo" parent_link="right_hand" x_origin="${-pinky_offset}"/>
+  <xacro:solenoid name="left_hand_thumb_solenoid" parent_link="left_hand_thumb_servo" />
+  <xacro:servo name="left_hand_thumb_servo" parent_link="left_hand" x_origin="${thumb_offset}" />
+  <xacro:solenoid name="left_hand_index_finger_solenoid" parent_link="left_hand_index_finger_servo" />
+  <xacro:servo name="left_hand_index_finger_servo" parent_link="left_hand"
+    x_origin="${index_offset}" />
+  <xacro:solenoid name="left_hand_middle_finger_solenoid"
+    parent_link="left_hand_middle_finger_servo" />
+  <xacro:servo name="left_hand_middle_finger_servo" parent_link="left_hand"
+    x_origin="${middle_offset}" />
+  <xacro:solenoid name="left_hand_ring_finger_solenoid" parent_link="left_hand_ring_finger_servo" />
+  <xacro:servo name="left_hand_ring_finger_servo" parent_link="left_hand" x_origin="${ring_offset}" />
+  <xacro:solenoid name="left_hand_pinky_solenoid" parent_link="left_hand_pinky_servo" />
+  <xacro:servo name="left_hand_pinky_servo" parent_link="left_hand" x_origin="${pinky_offset}" />
+  <xacro:solenoid name="right_hand_thumb_solenoid" parent_link="right_hand_thumb_servo" />
+  <xacro:servo name="right_hand_thumb_servo" parent_link="right_hand" x_origin="${-thumb_offset}" />
+  <xacro:solenoid name="right_hand_index_finger_solenoid"
+    parent_link="right_hand_index_finger_servo" />
+  <xacro:servo name="right_hand_index_finger_servo" parent_link="right_hand"
+    x_origin="${-index_offset}" />
+  <xacro:solenoid name="right_hand_middle_finger_solenoid"
+    parent_link="right_hand_middle_finger_servo" />
+  <xacro:servo name="right_hand_middle_finger_servo" parent_link="right_hand"
+    x_origin="${-middle_offset}" />
+  <xacro:solenoid name="right_hand_ring_finger_solenoid" parent_link="right_hand_ring_finger_servo" />
+  <xacro:servo name="right_hand_ring_finger_servo" parent_link="right_hand"
+    x_origin="${-ring_offset}" />
+  <xacro:solenoid name="right_hand_pinky_solenoid" parent_link="right_hand_pinky_servo" />
+  <xacro:servo name="right_hand_pinky_servo" parent_link="right_hand" x_origin="${-pinky_offset}" />
   <!-- Left Hand Fingers -->
-  <xacro:finger name="left_hand_thumb" parent_link="left_hand_thumb_solenoid"/>
-  <xacro:finger name="left_hand_index_finger" parent_link="left_hand_index_finger_solenoid"/>
-  <xacro:finger name="left_hand_middle_finger" parent_link="left_hand_middle_finger_solenoid"/>
-  <xacro:finger name="left_hand_ring_finger" parent_link="left_hand_ring_finger_solenoid"/>
-  <xacro:finger name="left_hand_pinky" parent_link="left_hand_pinky_solenoid"/>
+  <xacro:finger name="left_hand_thumb" parent_link="left_hand_thumb_solenoid" />
+  <xacro:finger name="left_hand_index_finger" parent_link="left_hand_index_finger_solenoid" />
+  <xacro:finger name="left_hand_middle_finger" parent_link="left_hand_middle_finger_solenoid" />
+  <xacro:finger name="left_hand_ring_finger" parent_link="left_hand_ring_finger_solenoid" />
+  <xacro:finger name="left_hand_pinky" parent_link="left_hand_pinky_solenoid" />
   <!-- Right Hand Fingers -->
-  <xacro:finger name="right_hand_thumb" parent_link="right_hand_thumb_solenoid"/>
-  <xacro:finger name="right_hand_index_finger" parent_link="right_hand_index_finger_solenoid"/>
-  <xacro:finger name="right_hand_middle_finger" parent_link="right_hand_middle_finger_solenoid"/>
-  <xacro:finger name="right_hand_ring_finger" parent_link="right_hand_ring_finger_solenoid"/>
-  <xacro:finger name="right_hand_pinky" parent_link="right_hand_pinky_solenoid"/>
+  <xacro:finger name="right_hand_thumb" parent_link="right_hand_thumb_solenoid" />
+  <xacro:finger name="right_hand_index_finger" parent_link="right_hand_index_finger_solenoid" />
+  <xacro:finger name="right_hand_middle_finger" parent_link="right_hand_middle_finger_solenoid" />
+  <xacro:finger name="right_hand_ring_finger" parent_link="right_hand_ring_finger_solenoid" />
+  <xacro:finger name="right_hand_pinky" parent_link="right_hand_pinky_solenoid" />
 </robot>
