Commit message: -Updated description and other stuff.

File: src/description/description/bothoven_core.xacro (robot description, xacro)
@@ -1,84 +1,73 @@
 <?xml version="1.0"?>
-<robot xmlns:xacro="http://www.ros.org/wiki/xacro">
-  <xacro:include filename="$(find description)/description/common.xacro" />
-  <!-- Robot Properties -->
+<robot name="bothoven" xmlns:xacro="http://www.ros.org/wiki/xacro">
+  <!-- Import hand macros -->
+  <xacro:include filename="$(find description)/description/left_hand.xacro" />
+  <xacro:include filename="$(find description)/description/right_hand.xacro" />
+  <!-- Rail properties -->
+  <xacro:property name="rail_length" value="1.2192" /> <!-- ~4 feet in meters -->
+  <xacro:property name="rail_width" value="0.05" />
+  <xacro:property name="rail_height" value="0.02" />
+  <!-- Define materials at the top level -->
+  <material name="servo_material">
+    <color rgba="0.302 0.314 0.8 1.0"/>
+  </material>
+  <!-- Dimensions -->
+  <xacro:property name="hand_width" value="0.2032" />
+  <xacro:property name="half_length" value="${rail_length / 2}" />
+  <xacro:property name="lh_start_point" value="-0.3" />
+  <xacro:property name="rh_start_point" value="0.3" />
+  <!-- Stepper consts -->
+  <xacro:property name="lh_stepper_min" value="${-(half_length + lh_start_point)}" />
+  <xacro:property name="lh_stepper_max" value="${half_length - lh_start_point - hand_width}" />
+  <xacro:property name="rh_stepper_min" value="${-(half_length + rh_start_point) + hand_width}" />
+  <xacro:property name="rh_stepper_max" value="${half_length - rh_start_point}" />
+  <!-- Solenoid Joint Properties -->
+  <xacro:property name="servo_min" value="-0.087266462599716473902" />
+  <xacro:property name="servo_max" value="0.087266462599716473902" />
+  <!-- Solenoid Joint Properties -->
+  <xacro:property name="solenoid_min" value="0" />
+  <xacro:property name="solenoid_max" value="0.52359877559829881566" />
+  <material name="finger_mount_plate_material">
+    <color rgba="0.231 0.380 0.706 1.0"/>
+  </material>
+  <material name="servo_mechanism_top_mount_material">
+    <color rgba="0.918 0.918 0.918 1.0"/>
+  </material>
+  <material name="large_solenoid_material">
+    <color rgba="0.980 0.714 0.004 1.0"/>
+  </material>
+  <material name="large_finger_solenoid_material">
+    <color rgba="0.769 0.886 0.953 1.0"/>
+  </material>
+  <material name="finger_arm_large_material">
+    <color rgba="0.973 0.529 0.004 1.0"/>
+  </material>
+  <material name="rail_material">
+    <color rgba="0.7 0.7 0.7 1.0"/>
+  </material>
+  <!-- Base link -->
   <link name="base_link">
+    <!-- Optional: Add a visual to represent the rail -->
+    <visual>
+      <origin xyz="0 0 0" rpy="0 0 0" />
+      <geometry>
+        <box size="0.01 ${rail_length} ${rail_height}"/>
+      </geometry>
+      <material name="rail_material"/>
+    </visual>
+    <collision>
+      <origin xyz="0 0 0" rpy="0 0 0" />
+      <geometry>
+        <box size="0.01 ${rail_length} ${rail_height}"/>
+      </geometry>
+    </collision>
     <inertial>
       <mass value="1.0" />
-      <origin xyz="0 0 0" />
       <inertia ixx="0.1" ixy="0.0" ixz="0.0" iyy="0.1" iyz="0.0" izz="0.1" />
     </inertial>
   </link>
-  <!-- Aluminum Rail -->
-  <link name="aluminum_rail">
-    <visual>
-      <geometry>
-        <box size="1.5 0.02 0.02" />
-      </geometry>
-      <material name="white" />
-    </visual>
-    <gazebo>
-      <material>Gazebo/White</material>
-    </gazebo>
-  </link>
-  <joint name="rail_to_base" type="fixed">
-    <parent link="base_link" />
-    <child link="aluminum_rail" />
-    <origin xyz="0 0 0.1" />
-    <gazebo>
-      <disableFixedJointLumping>false</disableFixedJointLumping>
-    </gazebo>
-  </joint>
-  <!-- Stepper Motors -->
-  <xacro:stepper name="left_hand_stepper" parent_link="aluminum_rail" origin_xyz="0.75 0 0" />
-  <xacro:stepper name="right_hand_stepper" parent_link="aluminum_rail" origin_xyz="-0.75 0 0" />
-  <!-- Carriages -->
-  <xacro:carriage name="left_carriage" parent_link="aluminum_rail" axis_x="-1"
-    mimic="left_hand_stepper_joint" />
-  <xacro:carriage name="right_carriage" parent_link="aluminum_rail" axis_x="1"
-    mimic="right_hand_stepper_joint" />
-  <!-- Hands -->
-  <xacro:hand name="left_hand" parent_link="left_carriage" />
-  <xacro:hand name="right_hand" parent_link="right_carriage" />
-  <!-- Solenoids and Servos attached to each finger -->
-  <xacro:solenoid name="left_hand_thumb_solenoid" parent_link="left_hand_thumb_servo" />
-  <xacro:servo name="left_hand_thumb_servo" parent_link="left_hand" x_origin="${thumb_offset}" />
-  <xacro:solenoid name="left_hand_index_finger_solenoid" parent_link="left_hand_index_finger_servo" />
-  <xacro:servo name="left_hand_index_finger_servo" parent_link="left_hand"
-    x_origin="${index_offset}" />
-  <xacro:solenoid name="left_hand_middle_finger_solenoid"
-    parent_link="left_hand_middle_finger_servo" />
-  <xacro:servo name="left_hand_middle_finger_servo" parent_link="left_hand"
-    x_origin="${middle_offset}" />
-  <xacro:solenoid name="left_hand_ring_finger_solenoid" parent_link="left_hand_ring_finger_servo" />
-  <xacro:servo name="left_hand_ring_finger_servo" parent_link="left_hand" x_origin="${ring_offset}" />
-  <xacro:solenoid name="left_hand_pinky_solenoid" parent_link="left_hand_pinky_servo" />
-  <xacro:servo name="left_hand_pinky_servo" parent_link="left_hand" x_origin="${pinky_offset}" />
-  <xacro:solenoid name="right_hand_thumb_solenoid" parent_link="right_hand_thumb_servo" />
-  <xacro:servo name="right_hand_thumb_servo" parent_link="right_hand" x_origin="${-thumb_offset}" />
-  <xacro:solenoid name="right_hand_index_finger_solenoid"
-    parent_link="right_hand_index_finger_servo" />
-  <xacro:servo name="right_hand_index_finger_servo" parent_link="right_hand"
-    x_origin="${-index_offset}" />
-  <xacro:solenoid name="right_hand_middle_finger_solenoid"
-    parent_link="right_hand_middle_finger_servo" />
-  <xacro:servo name="right_hand_middle_finger_servo" parent_link="right_hand"
-    x_origin="${-middle_offset}" />
-  <xacro:solenoid name="right_hand_ring_finger_solenoid" parent_link="right_hand_ring_finger_servo" />
-  <xacro:servo name="right_hand_ring_finger_servo" parent_link="right_hand"
-    x_origin="${-ring_offset}" />
-  <xacro:solenoid name="right_hand_pinky_solenoid" parent_link="right_hand_pinky_servo" />
-  <xacro:servo name="right_hand_pinky_servo" parent_link="right_hand" x_origin="${-pinky_offset}" />
-  <!-- Left Hand Fingers -->
-  <xacro:finger name="left_hand_thumb" parent_link="left_hand_thumb_solenoid" />
-  <xacro:finger name="left_hand_index_finger" parent_link="left_hand_index_finger_solenoid" />
-  <xacro:finger name="left_hand_middle_finger" parent_link="left_hand_middle_finger_solenoid" />
-  <xacro:finger name="left_hand_ring_finger" parent_link="left_hand_ring_finger_solenoid" />
-  <xacro:finger name="left_hand_pinky" parent_link="left_hand_pinky_solenoid" />
-  <!-- Right Hand Fingers -->
-  <xacro:finger name="right_hand_thumb" parent_link="right_hand_thumb_solenoid" />
-  <xacro:finger name="right_hand_index_finger" parent_link="right_hand_index_finger_solenoid" />
-  <xacro:finger name="right_hand_middle_finger" parent_link="right_hand_middle_finger_solenoid" />
-  <xacro:finger name="right_hand_ring_finger" parent_link="right_hand_ring_finger_solenoid" />
-  <xacro:finger name="right_hand_pinky" parent_link="right_hand_pinky_solenoid" />
+  <!-- Create left hand -->
+  <xacro:left_hand parent_link="base_link" rail_origin="0" rail_length="${rail_length}" />
+  <!-- Create right hand -->
+  <xacro:right_hand parent_link="base_link" rail_origin="0" rail_length="${rail_length}" />
 </robot>

File: src/hardware/urdf/left_servo_joints.xacro (robot description, xacro)
@@ -1,5 +1,5 @@
 <?xml version="1.0"?>
 <robot xmlns:xacro="http://www.ros.org/wiki/xacro">
-    <joint name="left_hand_thumb_servo_joint">
+    <joint name="lh_servo_1">
         <command_interface name="position">
             <param name="min">${servo_min}</param>
@@ -8,5 +8,5 @@
         <state_interface name="position" />
     </joint>
-    <joint name="left_hand_index_finger_servo_joint">
+    <joint name="lh_servo_2">
         <command_interface name="position">
             <param name="min">${servo_min}</param>
@@ -15,5 +15,5 @@
         <state_interface name="position" />
     </joint>
-    <joint name="left_hand_middle_finger_servo_joint">
+    <joint name="lh_servo_3">
         <command_interface name="position">
             <param name="min">${servo_min}</param>
@@ -22,5 +22,5 @@
         <state_interface name="position" />
     </joint>
-    <joint name="left_hand_ring_finger_servo_joint">
+    <joint name="lh_servo_4">
         <command_interface name="position">
             <param name="min">${servo_min}</param>
@@ -29,5 +29,5 @@
         <state_interface name="position" />
     </joint>
-    <joint name="left_hand_pinky_servo_joint">
+    <joint name="lh_servo_5">
         <command_interface name="position">
             <param name="min">${servo_min}</param>

File: src/hardware/urdf/left_solenoid_joints.xacro (robot description, xacro)
@@ -1,5 +1,5 @@
 <?xml version="1.0"?>
 <robot xmlns:xacro="http://www.ros.org/wiki/xacro">
-    <joint name="left_hand_thumb_solenoid_joint">
+    <joint name="lh_solenoid_1">
         <command_interface name="position">
             <param name="min">${solenoid_min}</param>
@@ -8,5 +8,5 @@
         <state_interface name="position" />
     </joint>
-    <joint name="left_hand_index_finger_solenoid_joint">
+    <joint name="lh_solenoid_2">
         <command_interface name="position">
             <param name="min">${solenoid_min}</param>
@@ -15,5 +15,5 @@
         <state_interface name="position" />
     </joint>
-    <joint name="left_hand_middle_finger_solenoid_joint">
+    <joint name="lh_solenoid_3">
         <command_interface name="position">
             <param name="min">${solenoid_min}</param>
@@ -22,5 +22,5 @@
         <state_interface name="position" />
     </joint>
-    <joint name="left_hand_ring_finger_solenoid_joint">
+    <joint name="lh_solenoid_4">
         <command_interface name="position">
             <param name="min">${solenoid_min}</param>
@@ -29,5 +29,5 @@
         <state_interface name="position" />
     </joint>
-    <joint name="left_hand_pinky_solenoid_joint">
+    <joint name="lh_solenoid_5">
         <command_interface name="position">
             <param name="min">${solenoid_min}</param>

File: src/hardware/urdf/left_stepper_joint.xacro (robot description, xacro)
@@ -1,8 +1,8 @@
 <?xml version="1.0"?>
 <robot xmlns:xacro="http://www.ros.org/wiki/xacro">
-    <joint name="left_hand_stepper_joint">
+    <joint name="lh_stepper">
         <command_interface name="position">
-            <param name="min">${stepper_min_angle}</param>
-            <param name="max">${stepper_max_angle}</param>
+            <param name="min">${lh_stepper_min}</param>
+            <param name="max">${lh_stepper_max}</param>
         </command_interface>
         <state_interface name="position" />

File: src/hardware/urdf/right_servo_joints.xacro (robot description, xacro)
@@ -1,5 +1,5 @@
 <?xml version="1.0"?>
 <robot xmlns:xacro="http://www.ros.org/wiki/xacro">
-    <joint name="right_hand_thumb_servo_joint">
+    <joint name="rh_servo_1">
         <command_interface name="position">
             <param name="min">${servo_min}</param>
@@ -8,5 +8,5 @@
         <state_interface name="position" />
     </joint>
-    <joint name="right_hand_index_finger_servo_joint">
+    <joint name="rh_servo_2">
         <command_interface name="position">
             <param name="min">${servo_min}</param>
@@ -15,5 +15,5 @@
         <state_interface name="position" />
     </joint>
-    <joint name="right_hand_middle_finger_servo_joint">
+    <joint name="rh_servo_3">
         <command_interface name="position">
             <param name="min">${servo_min}</param>
@@ -22,5 +22,5 @@
         <state_interface name="position" />
     </joint>
-    <joint name="right_hand_ring_finger_servo_joint">
+    <joint name="rh_servo_4">
         <command_interface name="position">
             <param name="min">${servo_min}</param>
@@ -29,5 +29,5 @@
         <state_interface name="position" />
     </joint>
-    <joint name="right_hand_pinky_servo_joint">
+    <joint name="rh_servo_5">
         <command_interface name="position">
             <param name="min">${servo_min}</param>

File: src/hardware/urdf/right_solenoid_joints.xacro (robot description, xacro)
@@ -1,5 +1,5 @@
 <?xml version="1.0"?>
 <robot xmlns:xacro="http://www.ros.org/wiki/xacro">
-    <joint name="right_hand_thumb_solenoid_joint">
+    <joint name="lh_solenoid_1">
         <command_interface name="position">
             <param name="min">${solenoid_min}</param>
@@ -8,5 +8,5 @@
         <state_interface name="position" />
     </joint>
-    <joint name="right_hand_index_finger_solenoid_joint">
+    <joint name="lh_solenoid_2">
         <command_interface name="position">
             <param name="min">${solenoid_min}</param>
@@ -15,5 +15,5 @@
         <state_interface name="position" />
     </joint>
-    <joint name="right_hand_middle_finger_solenoid_joint">
+    <joint name="lh_solenoid_3">
         <command_interface name="position">
             <param name="min">${solenoid_min}</param>
@@ -22,5 +22,5 @@
         <state_interface name="position" />
     </joint>
-    <joint name="right_hand_ring_finger_solenoid_joint">
+    <joint name="lh_solenoid_4">
         <command_interface name="position">
             <param name="min">${solenoid_min}</param>
@@ -29,5 +29,5 @@
         <state_interface name="position" />
     </joint>
-    <joint name="right_hand_pinky_solenoid_joint">
+    <joint name="lh_solenoid_5">
         <command_interface name="position">
             <param name="min">${solenoid_min}</param>

File: src/hardware/urdf/right_stepper_joint.xacro (robot description, xacro)
@@ -1,8 +1,8 @@
 <?xml version="1.0"?>
 <robot xmlns:xacro="http://www.ros.org/wiki/xacro">
-    <joint name="right_hand_stepper_joint">
+    <joint name="rh_stepper">
         <command_interface name="position">
-            <param name="min">${stepper_min_angle}</param>
-            <param name="max">${stepper_max_angle}</param>
+            <param name="min">${rh_stepper_min}</param>
+            <param name="max">${rh_stepper_max}</param>
         </command_interface>
         <state_interface name="position" />

File: src/hardware/urdf/ros2_control.xacro (robot description, xacro)
@@ -22,5 +22,5 @@
       <xacro:include filename="$(find hardware)/urdf/left_stepper_joint.xacro" />
     </ros2_control>
-    <ros2_control name="right_stepper_driver" type="system" is_async="false">
+    <!-- <ros2_control name="right_stepper_driver" type="system" is_async="false">
       <xacro:unless value="${use_mock_hardware}">
         <hardware>
@@ -41,5 +41,5 @@
       </xacro:if>
       <xacro:include filename="$(find hardware)/urdf/right_stepper_joint.xacro" />
-    </ros2_control>
+    </ros2_control> -->
     <ros2_control name="left_servo_driver" type="system">
       <xacro:unless value="${use_mock_hardware}">
@@ -48,5 +48,5 @@
           <param name="i2c_device">/dev/i2c-1</param>
           <param name="frequency_hz">50</param>
-          <param name="i2c_address">64</param>
+          <param name="i2c_address">65</param>
           <param name="min_duty_cycle_ms">1.3</param>
           <param name="max_duty_cycle_ms">1.7</param>
@@ -62,5 +62,5 @@
       <xacro:include filename="$(find hardware)/urdf/left_servo_joints.xacro" />
     </ros2_control>
-    <ros2_control name="right_servo_driver" type="system">
+    <!-- <ros2_control name="right_servo_driver" type="system">
       <xacro:unless value="${use_mock_hardware}">
         <hardware>
@@ -68,5 +68,5 @@
           <param name="i2c_device">/dev/i2c-1</param>
           <param name="frequency_hz">50</param>
-          <param name="i2c_address">65</param>
+          <param name="i2c_address">64</param>
           <param name="min_duty_cycle_ms">1.0</param>
           <param name="max_duty_cycle_ms">2.0</param>
@@ -81,6 +81,23 @@
       </xacro:if>
       <xacro:include filename="$(find hardware)/urdf/right_servo_joints.xacro" />
+    </ros2_control> -->
+    <ros2_control name="left_solenoid_driver" type="system">
+      <xacro:unless value="${use_mock_hardware}">
+        <hardware>
+          <plugin>mcp23017_hardware_interface/Mcp23017SystemHardware</plugin>
+          <param name="i2c_device">/dev/i2c-1</param>
+          <param name="i2c_address">33</param>
+        </hardware>
+      </xacro:unless>
+      <xacro:if value="${use_mock_hardware}">
+        <hardware>
+          <plugin>mock_components/GenericSystem</plugin>
+          <param name="calculate_dynamics">true</param>
+          <param name="mock_gpio_commands">true</param>
+        </hardware>
+      </xacro:if>
+      <xacro:include filename="$(find hardware)/urdf/left_solenoid_joints.xacro" />
     </ros2_control>
-    <ros2_control name="left_solenoid_driver" type="system">
+    <!-- <ros2_control name="right_solenoid_driver" type="system">
       <xacro:unless value="${use_mock_hardware}">
         <hardware>
@@ -97,23 +114,6 @@
         </hardware>
       </xacro:if>
-      <xacro:include filename="$(find hardware)/urdf/left_solenoid_joints.xacro" />
-    </ros2_control>
-    <ros2_control name="right_solenoid_driver" type="system">
-      <xacro:unless value="${use_mock_hardware}">
-        <hardware>
-          <plugin>mcp23017_hardware_interface/Mcp23017SystemHardware</plugin>
-          <param name="i2c_device">/dev/i2c-1</param>
-          <param name="i2c_address">33</param>
-        </hardware>
-      </xacro:unless>
-      <xacro:if value="${use_mock_hardware}">
-        <hardware>
-          <plugin>mock_components/GenericSystem</plugin>
-          <param name="calculate_dynamics">true</param>
-          <param name="mock_gpio_commands">true</param>
-        </hardware>
-      </xacro:if>
       <xacro:include filename="$(find hardware)/urdf/right_solenoid_joints.xacro" />
-    </ros2_control>
+    </ros2_control> -->
   </xacro:macro>
 </robot>
