Commit message: getting closer to the end.... steppers and servos need to work

File: src/description/description/finger.xacro (robot description, xacro)
@@ -8,5 +8,5 @@
         <origin xyz="0 0.027359073967098360841 -0.036000000000000004219" rpy="0 0 0" />
         <geometry>
-          <mesh filename="package://description/meshes/large_solenoid.stl"/>
+          <mesh filename="package://description/description/meshes/large_solenoid.stl"/>
         </geometry>
         <material name="large_solenoid_material"/>
@@ -15,5 +15,5 @@
         <origin xyz="1.3877787807814456755e-17 0.0074929958267665672245 0" rpy="3.141592653589793116 0 0" />
         <geometry>
-          <mesh filename="package://description/meshes/large_finger_solenoid.stl"/>
+          <mesh filename="package://description/description/meshes/large_finger_solenoid.stl"/>
         </geometry>
         <material name="large_finger_solenoid_material"/>
@@ -30,5 +30,5 @@
         <origin xyz="0.063368257669539254651 -5.4787295081876186131e-05 -0.0050000000000000044409" rpy="0 0 0" />
         <geometry>
-          <mesh filename="package://description/meshes/finger_arm_large.stl"/>
+          <mesh filename="package://description/description/meshes/finger_arm_large.stl"/>
         </geometry>
         <material name="finger_arm_large_material"/>

File: src/description/description/left_hand.xacro (robot description, xacro)
@@ -24,5 +24,5 @@
         <origin xyz="0.045938244354197944885 -0.043846468705386110187 0.078200000000000005618" rpy="3.141592653589793116 -0 3.141592653589793116" />
         <geometry>
-          <mesh filename="package://description/meshes/servo.stl"/>
+          <mesh filename="package://description/description/meshes/servo.stl"/>
         </geometry>
         <material name="servo_material"/>
@@ -31,5 +31,5 @@
         <origin xyz="0.045938244354197944885 -0.0063464687053861098404 0.078200000000000005618" rpy="3.141592653589793116 -0 3.141592653589793116" />
         <geometry>
-          <mesh filename="package://description/meshes/servo.stl"/>
+          <mesh filename="package://description/description/meshes/servo.stl"/>
         </geometry>
         <material name="servo_material"/>
@@ -38,5 +38,5 @@
         <origin xyz="0.0023499287608851338049 0.033803517640591265736 -0.021799999999999989525" rpy="1.9958838398273146999e-16 -6.5938365254384542654e-32 0" />
         <geometry>
-          <mesh filename="package://description/meshes/finger_mount_plate.stl"/>
+          <mesh filename="package://description/description/meshes/finger_mount_plate.stl"/>
         </geometry>
         <material name="finger_mount_plate_material"/>
@@ -45,5 +45,5 @@
         <origin xyz="0.045938244354197951824 0.068653531294613892588 0.078200000000000005618" rpy="3.141592653589793116 -0 3.141592653589793116" />
         <geometry>
-          <mesh filename="package://description/meshes/servo.stl"/>
+          <mesh filename="package://description/description/meshes/servo.stl"/>
         </geometry>
         <material name="servo_material"/>
@@ -52,5 +52,5 @@
         <origin xyz="0.045938244354197944885 0.031153531294613880098 0.078200000000000005618" rpy="3.141592653589793116 -0 3.141592653589793116" />
         <geometry>
-          <mesh filename="package://description/meshes/servo.stl"/>
+          <mesh filename="package://description/description/meshes/servo.stl"/>
         </geometry>
         <material name="servo_material"/>
@@ -59,5 +59,5 @@
         <origin xyz="0.002343270376630176427 3.5176405913106556511e-06 0.060000000000000004718" rpy="3.141592653589793116 -0 0" />
         <geometry>
-          <mesh filename="package://description/meshes/servo_mechanism_top_mount.stl"/>
+          <mesh filename="package://description/description/meshes/servo_mechanism_top_mount.stl"/>
         </geometry>
         <material name="servo_mechanism_top_mount_material"/>
@@ -66,5 +66,5 @@
         <origin xyz="0.045938244354197944885 -0.081346468705386101861 0.078200000000000005618" rpy="3.141592653589793116 -0 3.141592653589793116" />
         <geometry>
-          <mesh filename="package://description/meshes/servo.stl"/>
+          <mesh filename="package://description/description/meshes/servo.stl"/>
         </geometry>
         <material name="servo_material"/>

File: src/description/description/right_hand.xacro (robot description, xacro)
@@ -24,5 +24,5 @@
         <origin xyz="0.045938244354197944885 -0.043846468705386110187 0.078200000000000005618" rpy="3.141592653589793116 -0 3.141592653589793116" />
         <geometry>
-          <mesh filename="package://description/meshes/servo.stl"/>
+          <mesh filename="package://description/description/meshes/servo.stl"/>
         </geometry>
         <material name="servo_material"/>
@@ -31,5 +31,5 @@
         <origin xyz="0.045938244354197944885 -0.0063464687053861098404 0.078200000000000005618" rpy="3.141592653589793116 -0 3.141592653589793116" />
         <geometry>
-          <mesh filename="package://description/meshes/servo.stl"/>
+          <mesh filename="package://description/description/meshes/servo.stl"/>
         </geometry>
         <material name="servo_material"/>
@@ -38,5 +38,5 @@
         <origin xyz="0.0023499287608851338049 0.033803517640591265736 -0.021799999999999989525" rpy="1.9958838398273146999e-16 -6.5938365254384542654e-32 0" />
         <geometry>
-          <mesh filename="package://description/meshes/finger_mount_plate.stl"/>
+          <mesh filename="package://description/description/meshes/finger_mount_plate.stl"/>
         </geometry>
         <material name="finger_mount_plate_material"/>
@@ -45,5 +45,5 @@
         <origin xyz="0.045938244354197951824 0.068653531294613892588 0.078200000000000005618" rpy="3.141592653589793116 -0 3.141592653589793116" />
         <geometry>
-          <mesh filename="package://description/meshes/servo.stl"/>
+          <mesh filename="package://description/description/meshes/servo.stl"/>
         </geometry>
         <material name="servo_material"/>
@@ -52,5 +52,5 @@
         <origin xyz="0.045938244354197944885 0.031153531294613880098 0.078200000000000005618" rpy="3.141592653589793116 -0 3.141592653589793116" />
         <geometry>
-          <mesh filename="package://description/meshes/servo.stl"/>
+          <mesh filename="package://description/description/meshes/servo.stl"/>
         </geometry>
         <material name="servo_material"/>
@@ -59,5 +59,5 @@
         <origin xyz="0.002343270376630176427 3.5176405913106556511e-06 0.060000000000000004718" rpy="3.141592653589793116 -0 0" />
         <geometry>
-          <mesh filename="package://description/meshes/servo_mechanism_top_mount.stl"/>
+          <mesh filename="package://description/description/meshes/servo_mechanism_top_mount.stl"/>
         </geometry>
         <material name="servo_mechanism_top_mount_material"/>
@@ -66,5 +66,5 @@
         <origin xyz="0.045938244354197944885 -0.081346468705386101861 0.078200000000000005618" rpy="3.141592653589793116 -0 3.141592653589793116" />
         <geometry>
-          <mesh filename="package://description/meshes/servo.stl"/>
+          <mesh filename="package://description/description/meshes/servo.stl"/>
         </geometry>
         <material name="servo_material"/>

File: src/hardware/urdf/left_servo_joints.xacro (robot description, xacro)
@@ -1,4 +1,5 @@
 <?xml version="1.0"?>
 <robot xmlns:xacro="http://www.ros.org/wiki/xacro">
+    <!-- thumb -->
     <joint name="lh_servo_1">
         <command_interface name="position">
@@ -7,5 +8,16 @@
         </command_interface>
         <state_interface name="position" />
+        <!-- PCA9685 parameters -->
+        <param name="servo_channel">4</param>
+        <param name="pwm_min">500</param>
+        <param name="pwm_max">2500</param>
+        <param name="pwm_slope">13.10</param>
+        <param name="pwm_intercept">339.41</param>
+        <!-- ADS7138 parameters -->
+        <param name="adc_channel">4</param>
+        <param name="adc_slope">2.33</param>
+        <param name="adc_intercept">91.48</param>
     </joint>
+    <!-- index -->
     <joint name="lh_servo_2">
         <command_interface name="position">
@@ -14,5 +26,16 @@
         </command_interface>
         <state_interface name="position" />
+        <!-- PCA9685 parameters -->
+        <param name="servo_channel">3</param>
+        <param name="pwm_min">500</param>
+        <param name="pwm_max">2500</param>
+        <param name="pwm_slope">13.20</param>
+        <param name="pwm_intercept">319.56</param>
+        <!-- ADS7138 parameters -->
+        <param name="adc_channel">3</param>
+        <param name="adc_slope">2.33</param>
+        <param name="adc_intercept">85.52</param>
     </joint>
+    <!-- middle -->
     <joint name="lh_servo_3">
         <command_interface name="position">
@@ -21,5 +44,16 @@
         </command_interface>
         <state_interface name="position" />
+        <!-- PCA9685 parameters -->
+        <param name="servo_channel">2</param>
+        <param name="pwm_min">500</param>
+        <param name="pwm_max">2500</param>
+        <param name="pwm_slope">12.33</param>
+        <param name="pwm_intercept">306.41</param>
+        <!-- ADS7138 parameters -->
+        <param name="adc_channel">2</param>
+        <param name="adc_slope">2.27</param>
+        <param name="adc_intercept">83.03</param>
     </joint>
+    <!-- ring -->
     <joint name="lh_servo_4">
         <command_interface name="position">
@@ -28,5 +62,16 @@
         </command_interface>
         <state_interface name="position" />
+        <!-- PCA9685 parameters -->
+        <param name="servo_channel">1</param>
+        <param name="pwm_min">500</param>
+        <param name="pwm_max">2500</param>
+        <param name="pwm_slope">12.84</param>
+        <param name="pwm_intercept">287.44</param>
+        <!-- ADS7138 parameters -->
+        <param name="adc_channel">1</param>
+        <param name="adc_slope">2.53</param>
+        <param name="adc_intercept">88.97</param>
     </joint>
+    <!-- pinky -->
     <joint name="lh_servo_5">
         <command_interface name="position">
@@ -35,4 +80,14 @@
         </command_interface>
         <state_interface name="position" />
+        <!-- PCA9685 parameters -->
+        <param name="servo_channel">0</param>
+        <param name="pwm_min">500</param>
+        <param name="pwm_max">2500</param>
+        <param name="pwm_slope">12.14</param>
+        <param name="pwm_intercept">519.92</param>
+        <!-- ADS7138 parameters -->
+        <param name="adc_channel">0</param>
+        <param name="adc_slope">1.83</param>
+        <param name="adc_intercept">101.71</param>
     </joint>
 </robot>

File: src/hardware/urdf/right_servo_joints.xacro (robot description, xacro)
@@ -1,4 +1,5 @@
 <?xml version="1.0"?>
 <robot xmlns:xacro="http://www.ros.org/wiki/xacro">
+    <!-- thumb -->
     <joint name="rh_servo_1">
         <command_interface name="position">
@@ -7,5 +8,16 @@
         </command_interface>
         <state_interface name="position" />
+        <!-- PCA9685 parameters -->
+        <param name="servo_channel">0</param>
+        <param name="pwm_min">500</param>
+        <param name="pwm_max">2500</param>
+        <param name="pwm_slope">13.05</param>
+        <param name="pwm_intercept">352.17</param>
+        <!-- ADS7138 parameters -->
+        <param name="adc_channel">0</param>
+        <param name="adc_slope">2.36</param>
+        <param name="adc_intercept">90.82</param>
     </joint>
+    <!-- index -->
     <joint name="rh_servo_2">
         <command_interface name="position">
@@ -14,5 +26,16 @@
         </command_interface>
         <state_interface name="position" />
+        <!-- PCA9685 parameters -->
+        <param name="servo_channel">1</param>
+        <param name="pwm_min">500</param>
+        <param name="pwm_max">2500</param>
+        <param name="pwm_slope">12.78</param>
+        <param name="pwm_intercept">357.69</param>
+        <!-- ADS7138 parameters -->
+        <param name="adc_channel">1</param>
+        <param name="adc_slope">2.49</param>
+        <param name="adc_intercept">101.49</param>
     </joint>
+    <!-- middle -->
     <joint name="rh_servo_3">
         <command_interface name="position">
@@ -21,5 +44,16 @@
         </command_interface>
         <state_interface name="position" />
+        <!-- PCA9685 parameters -->
+        <param name="servo_channel">2</param>
+        <param name="pwm_min">500</param>
+        <param name="pwm_max">2500</param>
+        <param name="pwm_slope">12.96</param>
+        <param name="pwm_intercept">411.49</param>
+        <!-- ADS7138 parameters -->
+        <param name="adc_channel">2</param>
+        <param name="adc_slope">2.24</param>
+        <param name="adc_intercept">108.88</param>
     </joint>
+    <!-- ring -->
     <joint name="rh_servo_4">
         <command_interface name="position">
@@ -28,5 +62,16 @@
         </command_interface>
         <state_interface name="position" />
+        <!-- PCA9685 parameters -->
+        <param name="servo_channel">3</param>
+        <param name="pwm_min">500</param>
+        <param name="pwm_max">2500</param>
+        <param name="pwm_slope">12.51</param>
+        <param name="pwm_intercept">443.14</param>
+        <!-- ADS7138 parameters -->
+        <param name="adc_channel">3</param>
+        <param name="adc_slope">2.26</param>
+        <param name="adc_intercept">108.08</param>
     </joint>
+    <!-- pinky -->
     <joint name="rh_servo_5">
         <command_interface name="position">
@@ -35,4 +80,14 @@
         </command_interface>
         <state_interface name="position" />
+        <!-- PCA9685 parameters -->
+        <param name="servo_channel">4</param>
+        <param name="pwm_min">500</param>
+        <param name="pwm_max">2500</param>
+        <param name="pwm_slope">12.87</param>
+        <param name="pwm_intercept">372.07</param>
+        <!-- ADS7138 parameters -->
+        <param name="adc_channel">4</param>
+        <param name="adc_slope">2.29</param>
+        <param name="adc_intercept">97.49</param>
     </joint>
 </robot>

File: src/hardware/urdf/right_solenoid_joints.xacro (robot description, xacro)
@@ -1,5 +1,5 @@
 <?xml version="1.0"?>
 <robot xmlns:xacro="http://www.ros.org/wiki/xacro">
-    <joint name="lh_solenoid_1">
+    <joint name="rh_solenoid_1">
         <command_interface name="position">
             <param name="min">${solenoid_min}</param>
@@ -8,5 +8,5 @@
         <state_interface name="position" />
     </joint>
-    <joint name="lh_solenoid_2">
+    <joint name="rh_solenoid_2">
         <command_interface name="position">
             <param name="min">${solenoid_min}</param>
@@ -15,5 +15,5 @@
         <state_interface name="position" />
     </joint>
-    <joint name="lh_solenoid_3">
+    <joint name="rh_solenoid_3">
         <command_interface name="position">
             <param name="min">${solenoid_min}</param>
@@ -22,5 +22,5 @@
         <state_interface name="position" />
     </joint>
-    <joint name="lh_solenoid_4">
+    <joint name="rh_solenoid_4">
         <command_interface name="position">
             <param name="min">${solenoid_min}</param>
@@ -29,5 +29,5 @@
         <state_interface name="position" />
     </joint>
-    <joint name="lh_solenoid_5">
+    <joint name="rh_solenoid_5">
         <command_interface name="position">
             <param name="min">${solenoid_min}</param>

File: src/hardware/urdf/ros2_control.xacro (robot description, xacro)
@@ -22,5 +22,5 @@
       <xacro:include filename="$(find hardware)/urdf/left_stepper_joint.xacro" />
     </ros2_control>
-    <!-- <ros2_control name="right_stepper_driver" type="system" is_async="false">
+    <ros2_control name="right_stepper_driver" type="system" is_async="false">
       <xacro:unless value="${use_mock_hardware}">
         <hardware>
@@ -41,5 +41,5 @@
       </xacro:if>
       <xacro:include filename="$(find hardware)/urdf/right_stepper_joint.xacro" />
-    </ros2_control> -->
+    </ros2_control>
     <ros2_control name="left_servo_driver" type="system">
       <xacro:unless value="${use_mock_hardware}">
@@ -47,8 +47,10 @@
           <plugin>pca9685_hardware_interface/Pca9685SystemHardware</plugin>
           <param name="i2c_device">/dev/i2c-1</param>
-          <param name="frequency_hz">50</param>
-          <param name="i2c_address">65</param>
-          <param name="min_duty_cycle_ms">1.3</param>
-          <param name="max_duty_cycle_ms">1.7</param>
+          <param name="pca_frequency_hz">50</param>
+          <param name="pca_i2c_address">65</param>
+          <param name="min_duty_cycle_ms">0.5</param>
+          <param name="max_duty_cycle_ms">2.5</param>
+          <param name="ads_i2c_address">18</param> <!-- 0x10 -->
+          <param name="ads_conversion_rate">20</param> <!-- 20 kSPS -->
         </hardware>
       </xacro:unless>
@@ -62,13 +64,15 @@
       <xacro:include filename="$(find hardware)/urdf/left_servo_joints.xacro" />
     </ros2_control>
-    <!-- <ros2_control name="right_servo_driver" type="system">
+    <ros2_control name="right_servo_driver" type="system">
       <xacro:unless value="${use_mock_hardware}">
         <hardware>
           <plugin>pca9685_hardware_interface/Pca9685SystemHardware</plugin>
           <param name="i2c_device">/dev/i2c-1</param>
-          <param name="frequency_hz">50</param>
-          <param name="i2c_address">64</param>
-          <param name="min_duty_cycle_ms">1.0</param>
-          <param name="max_duty_cycle_ms">2.0</param>
+          <param name="pca_frequency_hz">50</param>
+          <param name="pca_i2c_address">64</param>
+          <param name="min_duty_cycle_ms">0.5</param>
+          <param name="max_duty_cycle_ms">2.5</param>
+          <param name="ads_i2c_address">16</param> <!-- 0x12 -->
+          <param name="ads_conversion_rate">20</param> <!-- 20 kSPS -->
         </hardware>
       </xacro:unless>
@@ -81,5 +85,5 @@
       </xacro:if>
       <xacro:include filename="$(find hardware)/urdf/right_servo_joints.xacro" />
-    </ros2_control> -->
+    </ros2_control>
     <ros2_control name="left_solenoid_driver" type="system">
       <xacro:unless value="${use_mock_hardware}">
@@ -99,5 +103,5 @@
       <xacro:include filename="$(find hardware)/urdf/left_solenoid_joints.xacro" />
     </ros2_control>
-    <!-- <ros2_control name="right_solenoid_driver" type="system">
+    <ros2_control name="right_solenoid_driver" type="system">
       <xacro:unless value="${use_mock_hardware}">
         <hardware>
@@ -115,5 +119,5 @@
       </xacro:if>
       <xacro:include filename="$(find hardware)/urdf/right_solenoid_joints.xacro" />
-    </ros2_control> -->
+    </ros2_control>
   </xacro:macro>
 </robot>
