Commit message: Updated URDF

File: src/description/urdf/bothoven.urdf.xacro (robot description, xacro)
@@ -46,5 +46,5 @@
   </link>
   <!-- Joints for hand movement on rails (using stepper motors) -->
-  <joint name="left_hand_to_left_rail" type="prismatic">
+  <joint name="left_hand_stepper_joint" type="prismatic">
     <parent link="left_rail"/>
     <child link="left_hand"/>
@@ -53,5 +53,5 @@
     <limit lower="0.0" upper="0.5" effort="5" velocity="1.0"/>
   </joint>
-  <joint name="right_hand_to_right_rail" type="prismatic">
+  <joint name="left_hand_stepper_joint" type="prismatic">
     <parent link="right_rail"/>
     <child link="right_hand"/>
@@ -161,49 +161,9 @@
       <param name="example_param">value</param>
     </hardware>
-    <joint name="left_hand_to_left_rail">
-      <command_interface name="position"/>
-      <state_interface name="position"/>
-    </joint>
-    <joint name="right_hand_to_right_rail">
-      <command_interface name="position"/>
-      <state_interface name="position"/>
-    </joint>
-    <joint name="left_hand_thumb_joint">
-      <command_interface name="position"/>
-      <state_interface name="position"/>
-    </joint>
-    <joint name="left_hand_index_finger_joint">
-      <command_interface name="position"/>
-      <state_interface name="position"/>
-    </joint>
-    <joint name="left_hand_middle_finger_joint">
-      <command_interface name="position"/>
-      <state_interface name="position"/>
-    </joint>
-    <joint name="left_hand_ring_finger_joint">
-      <command_interface name="position"/>
-      <state_interface name="position"/>
-    </joint>
-    <joint name="left_hand_pinky_joint">
-      <command_interface name="position"/>
-      <state_interface name="position"/>
-    </joint>
-    <joint name="right_hand_thumb_joint">
-      <command_interface name="position"/>
-      <state_interface name="position"/>
-    </joint>
-    <joint name="right_hand_index_finger_joint">
-      <command_interface name="position"/>
-      <state_interface name="position"/>
-    </joint>
-    <joint name="right_hand_middle_finger_joint">
-      <command_interface name="position"/>
-      <state_interface name="position"/>
-    </joint>
-    <joint name="right_hand_ring_finger_joint">
-      <command_interface name="position"/>
-      <state_interface name="position"/>
-    </joint>
-    <joint name="right_hand_pinky_joint">
+    <joint name="left_hand_stepper_joint">
+      <command_interface name="position"/>
+      <state_interface name="position"/>
+    </joint>
+    <joint name="left_hand_stepper_joint">
       <command_interface name="position"/>
       <state_interface name="position"/>

Commit message: Fixed URDF

File: src/description/urdf/bothoven.urdf.xacro (robot description, xacro)
@@ -2,27 +2,6 @@
 <robot name="bothoven" xmlns:xacro="http://www.ros.org/wiki/xacro">
   <!-- Robot Properties -->
-  <link name="world"/>
-  <!-- Rails and Hands -->
-  <link name="left_rail">
-    <visual>
-      <geometry>
-        <box size="0.5 0.1 0.05"/>
-      </geometry>
-      <material name="gray">
-        <color rgba="0.5 0.5 0.5 1.0"/>
-      </material>
-    </visual>
-  </link>
-  <link name="right_rail">
-    <visual>
-      <geometry>
-        <box size="0.5 0.1 0.05"/>
-      </geometry>
-      <material name="gray">
-        <color rgba="0.5 0.5 0.5 1.0"/>
-      </material>
-    </visual>
-  </link>
-  <!-- Define the hands (connected to rails via joints) -->
+  <link name="bothoven"/>
+    <!-- Define the hands (connected to rail via joints) -->
   <link name="left_hand">
     <visual>
@@ -47,5 +26,5 @@
   <!-- Joints for hand movement on rails (using stepper motors) -->
   <joint name="left_hand_stepper_joint" type="prismatic">
-    <parent link="left_rail"/>
+    <parent link="bothoven"/>
     <child link="left_hand"/>
     <origin xyz="0 0 0.05"/>
@@ -53,6 +32,6 @@
     <limit lower="0.0" upper="0.5" effort="5" velocity="1.0"/>
   </joint>
-  <joint name="left_hand_stepper_joint" type="prismatic">
-    <parent link="right_rail"/>
+  <joint name="right_hand_stepper_joint" type="prismatic">
+    <parent link="bothoven"/>
     <child link="right_hand"/>
     <origin xyz="0 0 0.05"/>
@@ -63,5 +42,4 @@
   <xacro:property name="finger_length" value="0.03"/>
   <xacro:property name="finger_thickness" value="0.01"/>
-  <!-- Left Hand Fingers -->
   <xacro:macro name="finger" params="name parent_link">
     <link name="${name}">
@@ -75,12 +53,11 @@
       </visual>
     </link>
-    <joint name="${name}_joint" type="revolute">
+    <joint name="${name}_joint" type="fixed">
       <parent link="${parent_link}"/>
       <child link="${name}"/>
-      <origin xyz="0 0 -0.05"/>
-      <axis xyz="0 1 0"/>
-      <limit lower="0" upper="1.57" effort="1" velocity="1.0"/>
+      <origin xyz="0 0 0"/>
     </joint>
   </xacro:macro>
+  <!-- Left Hand Fingers -->
   <xacro:finger name="left_hand_thumb" parent_link="left_hand"/>
   <xacro:finger name="left_hand_index_finger" parent_link="left_hand"/>
@@ -155,98 +132,3 @@
   <xacro:solenoid name="right_hand_pinky_solenoid" parent_link="right_hand_pinky"/>
   <xacro:servo name="right_hand_pinky_servo" parent_link="right_hand_pinky"/>
-  <!-- ros2_control Configuration -->
-  <ros2_control name="BothovenHardware" type="system">
-    <hardware>
-      <plugin>ros2_control_demo_hardware/GenericSystem</plugin>
-      <param name="example_param">value</param>
-    </hardware>
-    <joint name="left_hand_stepper_joint">
-      <command_interface name="position"/>
-      <state_interface name="position"/>
-    </joint>
-    <joint name="left_hand_stepper_joint">
-      <command_interface name="position"/>
-      <state_interface name="position"/>
-    </joint>
-    <joint name="left_hand_thumb_solenoid_joint">
-      <command_interface name="position"/>
-      <state_interface name="position"/>
-    </joint>
-    <joint name="left_hand_index_finger_solenoid_joint">
-      <command_interface name="position"/>
-      <state_interface name="position"/>
-    </joint>
-    <joint name="left_hand_middle_finger_solenoid_joint">
-      <command_interface name="position"/>
-      <state_interface name="position"/>
-    </joint>
-    <joint name="left_hand_ring_finger_solenoid_joint">
-      <command_interface name="position"/>
-      <state_interface name="position"/>
-    </joint>
-    <joint name="left_hand_pinky_solenoid_joint">
-      <command_interface name="position"/>
-      <state_interface name="position"/>
-    </joint>
-    <joint name="right_hand_thumb_solenoid_joint">
-      <command_interface name="position"/>
-      <state_interface name="position"/>
-    </joint>
-    <joint name="right_hand_index_finger_solenoid_joint">
-      <command_interface name="position"/>
-      <state_interface name="position"/>
-    </joint>
-    <joint name="right_hand_middle_finger_solenoid_joint">
-      <command_interface name="position"/>
-      <state_interface name="position"/>
-    </joint>
-    <joint name="right_hand_ring_finger_solenoid_joint">
-      <command_interface name="position"/>
-      <state_interface name="position"/>
-    </joint>
-    <joint name="right_hand_pinky_solenoid_joint">
-      <command_interface name="position"/>
-      <state_interface name="position"/>
-    </joint>
-    <joint name="left_hand_thumb_servo_joint">
-      <command_interface name="position"/>
-      <state_interface name="position"/>
-    </joint>
-    <joint name="left_hand_index_finger_servo_joint">
-      <command_interface name="position"/>
-      <state_interface name="position"/>
-    </joint>
-    <joint name="left_hand_middle_finger_servo_joint">
-      <command_interface name="position"/>
-      <state_interface name="position"/>
-    </joint>
-    <joint name="left_hand_ring_finger_servo_joint">
-      <command_interface name="position"/>
-      <state_interface name="position"/>
-    </joint>
-    <joint name="left_hand_pinky_servo_joint">
-      <command_interface name="position"/>
-      <state_interface name="position"/>
-    </joint>
-    <joint name="right_hand_thumb_servo_joint">
-      <command_interface name="position"/>
-      <state_interface name="position"/>
-    </joint>
-    <joint name="right_hand_index_finger_servo_joint">
-      <command_interface name="position"/>
-      <state_interface name="position"/>
-    </joint>
-    <joint name="right_hand_middle_finger_servo_joint">
-      <command_interface name="position"/>
-      <state_interface name="position"/>
-    </joint>
-    <joint name="right_hand_ring_finger_servo_joint">
-      <command_interface name="position"/>
-      <state_interface name="position"/>
-    </joint>
-    <joint name="right_hand_pinky_servo_joint">
-      <command_interface name="position"/>
-      <state_interface name="position"/>
-    </joint>
-  </ros2_control>
 </robot>

Commit message: Added the ros2_control description back

File: src/description/urdf/bothoven.urdf.xacro (robot description, xacro)
@@ -132,3 +132,98 @@
   <xacro:solenoid name="right_hand_pinky_solenoid" parent_link="right_hand_pinky"/>
   <xacro:servo name="right_hand_pinky_servo" parent_link="right_hand_pinky"/>
+  <!-- ros2_control Configuration -->
+  <ros2_control name="BothovenHardware" type="system">
+    <hardware>
+      <plugin>ros2_control_demo_hardware/GenericSystem</plugin>
+      <param name="example_param">value</param>
+    </hardware>
+    <joint name="left_hand_stepper_joint">
+      <command_interface name="position"/>
+      <state_interface name="position"/>
+    </joint>
+    <joint name="left_hand_stepper_joint">
+      <command_interface name="position"/>
+      <state_interface name="position"/>
+    </joint>
+    <joint name="left_hand_thumb_solenoid_joint">
+      <command_interface name="position"/>
+      <state_interface name="position"/>
+    </joint>
+    <joint name="left_hand_index_finger_solenoid_joint">
+      <command_interface name="position"/>
+      <state_interface name="position"/>
+    </joint>
+    <joint name="left_hand_middle_finger_solenoid_joint">
+      <command_interface name="position"/>
+      <state_interface name="position"/>
+    </joint>
+    <joint name="left_hand_ring_finger_solenoid_joint">
+      <command_interface name="position"/>
+      <state_interface name="position"/>
+    </joint>
+    <joint name="left_hand_pinky_solenoid_joint">
+      <command_interface name="position"/>
+      <state_interface name="position"/>
+    </joint>
+    <joint name="right_hand_thumb_solenoid_joint">
+      <command_interface name="position"/>
+      <state_interface name="position"/>
+    </joint>
+    <joint name="right_hand_index_finger_solenoid_joint">
+      <command_interface name="position"/>
+      <state_interface name="position"/>
+    </joint>
+    <joint name="right_hand_middle_finger_solenoid_joint">
+      <command_interface name="position"/>
+      <state_interface name="position"/>
+    </joint>
+    <joint name="right_hand_ring_finger_solenoid_joint">
+      <command_interface name="position"/>
+      <state_interface name="position"/>
+    </joint>
+    <joint name="right_hand_pinky_solenoid_joint">
+      <command_interface name="position"/>
+      <state_interface name="position"/>
+    </joint>
+    <joint name="left_hand_thumb_servo_joint">
+      <command_interface name="position"/>
+      <state_interface name="position"/>
+    </joint>
+    <joint name="left_hand_index_finger_servo_joint">
+      <command_interface name="position"/>
+      <state_interface name="position"/>
+    </joint>
+    <joint name="left_hand_middle_finger_servo_joint">
+      <command_interface name="position"/>
+      <state_interface name="position"/>
+    </joint>
+    <joint name="left_hand_ring_finger_servo_joint">
+      <command_interface name="position"/>
+      <state_interface name="position"/>
+    </joint>
+    <joint name="left_hand_pinky_servo_joint">
+      <command_interface name="position"/>
+      <state_interface name="position"/>
+    </joint>
+    <joint name="right_hand_thumb_servo_joint">
+      <command_interface name="position"/>
+      <state_interface name="position"/>
+    </joint>
+    <joint name="right_hand_index_finger_servo_joint">
+      <command_interface name="position"/>
+      <state_interface name="position"/>
+    </joint>
+    <joint name="right_hand_middle_finger_servo_joint">
+      <command_interface name="position"/>
+      <state_interface name="position"/>
+    </joint>
+    <joint name="right_hand_ring_finger_servo_joint">
+      <command_interface name="position"/>
+      <state_interface name="position"/>
+    </joint>
+    <joint name="right_hand_pinky_servo_joint">
+      <command_interface name="position"/>
+      <state_interface name="position"/>
+    </joint>
+  </ros2_control>
 </robot>

Commit message: Refactored URDF

File: src/description/urdf/bothoven.urdf.xacro (robot description, xacro)
@@ -1,229 +1,5 @@
 <?xml version="1.0"?>
 <robot name="bothoven" xmlns:xacro="http://www.ros.org/wiki/xacro">
-  <!-- Robot Properties -->
-  <link name="bothoven"/>
-    <!-- Define the hands (connected to rail via joints) -->
-  <link name="left_hand">
-    <visual>
-      <geometry>
-        <box size="0.1 0.05 0.05"/>
-      </geometry>
-      <material name="blue">
-        <color rgba="0.0 0.0 1.0 1.0"/>
-      </material>
-    </visual>
-  </link>
-  <link name="right_hand">
-    <visual>
-      <geometry>
-        <box size="0.1 0.05 0.05"/>
-      </geometry>
-      <material name="blue">
-        <color rgba="0.0 0.0 1.0 1.0"/>
-      </material>
-    </visual>
-  </link>
-  <!-- Joints for hand movement on rails (using stepper motors) -->
-  <joint name="left_hand_stepper_joint" type="prismatic">
-    <parent link="bothoven"/>
-    <child link="left_hand"/>
-    <origin xyz="0 0 0.05"/>
-    <axis xyz="1 0 0"/>
-    <limit lower="0.0" upper="0.5" effort="5" velocity="1.0"/>
-  </joint>
-  <joint name="right_hand_stepper_joint" type="prismatic">
-    <parent link="bothoven"/>
-    <child link="right_hand"/>
-    <origin xyz="0 0 0.05"/>
-    <axis xyz="1 0 0"/>
-    <limit lower="0.0" upper="0.5" effort="5" velocity="1.0"/>
-  </joint>
-  <!-- Fingers -->
-  <xacro:property name="finger_length" value="0.03"/>
-  <xacro:property name="finger_thickness" value="0.01"/>
-  <xacro:macro name="finger" params="name parent_link">
-    <link name="${name}">
-      <visual>
-        <geometry>
-          <box size="${finger_length} ${finger_thickness} ${finger_thickness}"/>
-        </geometry>
-        <material name="red">
-          <color rgba="1.0 0.0 0.0 1.0"/>
-        </material>
-      </visual>
-    </link>
-    <joint name="${name}_joint" type="fixed">
-      <parent link="${parent_link}"/>
-      <child link="${name}"/>
-      <origin xyz="0 0 0"/>
-    </joint>
-  </xacro:macro>
-  <!-- Left Hand Fingers -->
-  <xacro:finger name="left_hand_thumb" parent_link="left_hand"/>
-  <xacro:finger name="left_hand_index_finger" parent_link="left_hand"/>
-  <xacro:finger name="left_hand_middle_finger" parent_link="left_hand"/>
-  <xacro:finger name="left_hand_ring_finger" parent_link="left_hand"/>
-  <xacro:finger name="left_hand_pinky" parent_link="left_hand"/>
-  <!-- Right Hand Fingers -->
-  <xacro:finger name="right_hand_thumb" parent_link="right_hand"/>
-  <xacro:finger name="right_hand_index_finger" parent_link="right_hand"/>
-  <xacro:finger name="right_hand_middle_finger" parent_link="right_hand"/>
-  <xacro:finger name="right_hand_ring_finger" parent_link="right_hand"/>
-  <xacro:finger name="right_hand_pinky" parent_link="right_hand"/>
-  <!-- Solenoids for Finger Press -->
-  <xacro:macro name="solenoid" params="name parent_link">
-    <link name="${name}">
-      <visual>
-        <geometry>
-          <cylinder radius="0.01" length="0.02"/>
-        </geometry>
-        <material name="green">
-          <color rgba="0.0 1.0 0.0 1.0"/>
-        </material>
-      </visual>
-    </link>
-    <joint name="${name}_joint" type="prismatic">
-      <parent link="${parent_link}"/>
-      <child link="${name}"/>
-      <origin xyz="0 0 -0.01"/>
-      <axis xyz="0 0 1"/>
-      <limit lower="0" upper="0.01" effort="1" velocity="1.0"/>
-    </joint>
-  </xacro:macro>
-  <!-- Servos for Lateral Motion -->
-  <xacro:macro name="servo" params="name parent_link">
-    <link name="${name}">
-      <visual>
-        <geometry>
-          <box size="0.02 0.02 0.02"/>
-        </geometry>
-        <material name="yellow">
-          <color rgba="1.0 1.0 0.0 1.0"/>
-        </material>
-      </visual>
-    </link>
-    <joint name="${name}_joint" type="revolute">
-      <parent link="${parent_link}"/>
-      <child link="${name}"/>
-      <origin xyz="0 0 0"/>
-      <axis xyz="0 1 0"/>
-      <limit lower="-1.57" upper="1.57" effort="1" velocity="1.0"/>
-    </joint>
-  </xacro:macro>
-  <!-- Solenoids and Servos attached to each finger for key press and lateral motion -->
-  <xacro:solenoid name="left_hand_thumb_solenoid" parent_link="left_hand_thumb"/>
-  <xacro:servo name="left_hand_thumb_servo" parent_link="left_hand_thumb"/>
-  <xacro:solenoid name="left_hand_index_finger_solenoid" parent_link="left_hand_index_finger"/>
-  <xacro:servo name="left_hand_index_finger_servo" parent_link="left_hand_index_finger"/>
-  <xacro:solenoid name="left_hand_middle_finger_solenoid" parent_link="left_hand_middle_finger"/>
-  <xacro:servo name="left_hand_middle_finger_servo" parent_link="left_hand_middle_finger"/>
-  <xacro:solenoid name="left_hand_ring_finger_solenoid" parent_link="left_hand_ring_finger"/>
-  <xacro:servo name="left_hand_ring_finger_servo" parent_link="left_hand_ring_finger"/>
-  <xacro:solenoid name="left_hand_pinky_solenoid" parent_link="left_hand_pinky"/>
-  <xacro:servo name="left_hand_pinky_servo" parent_link="left_hand_pinky"/>
-  <xacro:solenoid name="right_hand_thumb_solenoid" parent_link="right_hand_thumb"/>
-  <xacro:servo name="right_hand_thumb_servo" parent_link="right_hand_thumb"/>
-  <xacro:solenoid name="right_hand_index_finger_solenoid" parent_link="right_hand_index_finger"/>
-  <xacro:servo name="right_hand_index_finger_servo" parent_link="right_hand_index_finger"/>
-  <xacro:solenoid name="right_hand_middle_finger_solenoid" parent_link="right_hand_middle_finger"/>
-  <xacro:servo name="right_hand_middle_finger_servo" parent_link="right_hand_middle_finger"/>
-  <xacro:solenoid name="right_hand_ring_finger_solenoid" parent_link="right_hand_ring_finger"/>
-  <xacro:servo name="right_hand_ring_finger_servo" parent_link="right_hand_ring_finger"/>
-  <xacro:solenoid name="right_hand_pinky_solenoid" parent_link="right_hand_pinky"/>
-  <xacro:servo name="right_hand_pinky_servo" parent_link="right_hand_pinky"/>
-  <!-- ros2_control Configuration -->
-  <ros2_control name="BothovenHardware" type="system">
-    <hardware>
-      <plugin>ros2_control_demo_hardware/GenericSystem</plugin>
-      <param name="example_param">value</param>
-    </hardware>
-    <joint name="left_hand_stepper_joint">
-      <command_interface name="position"/>
-      <state_interface name="position"/>
-    </joint>
-    <joint name="left_hand_stepper_joint">
-      <command_interface name="position"/>
-      <state_interface name="position"/>
-    </joint>
-    <joint name="left_hand_thumb_solenoid_joint">
-      <command_interface name="position"/>
-      <state_interface name="position"/>
-    </joint>
-    <joint name="left_hand_index_finger_solenoid_joint">
-      <command_interface name="position"/>
-      <state_interface name="position"/>
-    </joint>
-    <joint name="left_hand_middle_finger_solenoid_joint">
-      <command_interface name="position"/>
-      <state_interface name="position"/>
-    </joint>
-    <joint name="left_hand_ring_finger_solenoid_joint">
-      <command_interface name="position"/>
-      <state_interface name="position"/>
-    </joint>
-    <joint name="left_hand_pinky_solenoid_joint">
-      <command_interface name="position"/>
-      <state_interface name="position"/>
-    </joint>
-    <joint name="right_hand_thumb_solenoid_joint">
-      <command_interface name="position"/>
-      <state_interface name="position"/>
-    </joint>
-    <joint name="right_hand_index_finger_solenoid_joint">
-      <command_interface name="position"/>
-      <state_interface name="position"/>
-    </joint>
-    <joint name="right_hand_middle_finger_solenoid_joint">
-      <command_interface name="position"/>
-      <state_interface name="position"/>
-    </joint>
-    <joint name="right_hand_ring_finger_solenoid_joint">
-      <command_interface name="position"/>
-      <state_interface name="position"/>
-    </joint>
-    <joint name="right_hand_pinky_solenoid_joint">
-      <command_interface name="position"/>
-      <state_interface name="position"/>
-    </joint>
-    <joint name="left_hand_thumb_servo_joint">
-      <command_interface name="position"/>
-      <state_interface name="position"/>
-    </joint>
-    <joint name="left_hand_index_finger_servo_joint">
-      <command_interface name="position"/>
-      <state_interface name="position"/>
-    </joint>
-    <joint name="left_hand_middle_finger_servo_joint">
-      <command_interface name="position"/>
-      <state_interface name="position"/>
-    </joint>
-    <joint name="left_hand_ring_finger_servo_joint">
-      <command_interface name="position"/>
-      <state_interface name="position"/>
-    </joint>
-    <joint name="left_hand_pinky_servo_joint">
-      <command_interface name="position"/>
-      <state_interface name="position"/>
-    </joint>
-    <joint name="right_hand_thumb_servo_joint">
-      <command_interface name="position"/>
-      <state_interface name="position"/>
-    </joint>
-    <joint name="right_hand_index_finger_servo_joint">
-      <command_interface name="position"/>
-      <state_interface name="position"/>
-    </joint>
-    <joint name="right_hand_middle_finger_servo_joint">
-      <command_interface name="position"/>
-      <state_interface name="position"/>
-    </joint>
-    <joint name="right_hand_ring_finger_servo_joint">
-      <command_interface name="position"/>
-      <state_interface name="position"/>
-    </joint>
-    <joint name="right_hand_pinky_servo_joint">
-      <command_interface name="position"/>
-      <state_interface name="position"/>
-    </joint>
-  </ros2_control>
+  <xacro:include filename="./../description/bothoven_core.xacro"/>
+  <xacro:include filename="./../description/ros2_control.xacro"/>
 </robot>
