Commit message: start hardware refactor

File: src/bothoven_description/ros2_control/left_stepper_joint.xacro (robot description, xacro)
@@ -3,8 +3,6 @@
     <joint name="lh_stepper">
         <command_interface name="position">
-            <!-- <param name="min">${lh_stepper_min}</param>
-            <param name="max">${lh_stepper_max}</param> -->
-            <param name="min">0.000</param>
-            <param name="max">0.900</param>
+            <param name="min">${left_stepper_min}</param>
+            <param name="max">${left_stepper_max}</param>
         </command_interface>
         <state_interface name="position" />

File: src/bothoven_description/ros2_control/right_stepper_joint.xacro (robot description, xacro)
@@ -3,8 +3,6 @@
     <joint name="rh_stepper">
         <command_interface name="position">
-            <!-- <param name="min">${rh_stepper_min}</param>
-            <param name="max">${rh_stepper_max}</param> -->
-            <param name="min">0.000</param>
-            <param name="max">0.900</param>
+            <param name="min">${right_stepper_min}</param>
+            <param name="max">${right_stepper_max}</param>
         </command_interface>
         <state_interface name="position" />

File: src/bothoven_description/ros2_control/ros2_control.xacro (robot description, xacro)
@@ -13,8 +13,7 @@
           <param name="spi_device">/dev/spidev0.0</param>
           <param name="spi_mode">1</param>
-          <param name="bus_speed_hz">1000000</param>
+          <param name="bus_speed_hz">500000</param>
           <param name="bits_per_word">8</param>
           <param name="stepper_side">l</param>
-          <param name="max_position_error">0.002</param>
         </hardware>
       </xacro:unless>
@@ -35,5 +34,4 @@
           <param name="bits_per_word">8</param>
           <param name="stepper_side">r</param>
-          <param name="max_position_error">0.002</param>
         </hardware>
       </xacro:unless>
@@ -54,6 +52,6 @@
           <param name="min_duty_cycle_ms">0.5</param>
           <param name="max_duty_cycle_ms">2.5</param>
-          <param name="ads_i2c_address">16</param>          <!-- 0x10 -->
-          <param name="ads_conversion_rate">20</param>          <!-- 20 kSPS -->
+          <param name="ads_i2c_address">16</param>      <!-- 0x10 -->
+          <param name="ads_conversion_rate">20</param>  <!-- 20 kSPS -->
         </hardware>
       </xacro:unless>

File: src/bothoven_description/urdf/bothoven_core.xacro (robot description, xacro)
@@ -19,25 +19,30 @@
   <xacro:property name="solenoid_min" value="0" />
   <xacro:property name="solenoid_max" value="0.52359877559829881566" />
+  <!-- stepper joint limits -->
+  <xacro:property name="left_stepper_min" value="${-(rail_length/2 + lh_start_point)}" />
+  <xacro:property name="left_stepper_max" value="${rail_length/2 - lh_start_point - hand_width/2}" />
+  <xacro:property name="right_stepper_min" value="${-(rail_length/2 + rh_start_point) + hand_width/2}" />
+  <xacro:property name="right_stepper_max" value="${rail_length/2 - rh_start_point}" />
   <!-- colours -->
   <material name="finger_mount_plate_material">
-    <color rgba="0.231 0.380 0.706 1.0"/>
+    <color rgba="0.231 0.380 0.706 1.0" />
   </material>
   <material name="servo_mechanism_top_mount_material">
-    <color rgba="0.250 0.250 0.250 1.0"/>
+    <color rgba="0.250 0.250 0.250 1.0" />
   </material>
   <material name="servo_material">
-    <color rgba="0.302 0.314 0.8 1.0"/>
+    <color rgba="0.302 0.314 0.8 1.0" />
   </material>
   <material name="large_solenoid_material">
-    <color rgba="0.980 0.714 0.004 1.0"/>
+    <color rgba="0.980 0.714 0.004 1.0" />
   </material>
   <material name="large_finger_solenoid_material">
-    <color rgba="0.769 0.886 0.953 1.0"/>
+    <color rgba="0.769 0.886 0.953 1.0" />
   </material>
   <material name="finger_arm_large_material">
-    <color rgba="0.973 0.529 0.004 1.0"/>
+    <color rgba="0.973 0.529 0.004 1.0" />
   </material>
   <material name="rail_material">
-    <color rgba="0.7 0.7 0.7 1.0"/>
+    <color rgba="0.7 0.7 0.7 1.0" />
   </material>
   <!-- robot base -->
@@ -46,22 +51,32 @@
       <origin xyz="0 0 0" rpy="0 0 0" />
       <geometry>
-        <box size="0.01 ${rail_length} ${rail_height}"/>
+        <box size="0.01 ${rail_length} ${rail_height}" />
       </geometry>
-      <material name="rail_material"/>
+      <material name="rail_material" />
     </visual>
     <collision>
       <origin xyz="0 0 0" rpy="0 0 0" />
       <geometry>
-        <box size="0.01 ${rail_length} ${rail_height}"/>
+        <box size="0.01 ${rail_length} ${rail_height}" />
       </geometry>
+      <surface>
+        <friction>
+          <ode>
+            <mu>0.0</mu>
+            <mu2>0.0</mu2>
+          </ode>
+        </friction>
+      </surface>
     </collision>
     <inertial>
-      <origin xyz="0 0 0" rpy="0 0 0"/>
-      <mass value="10.0"/>
-      <inertia ixx="0.1" ixy="0.0" ixz="0.0" iyy="0.1" iyz="0.0" izz="0.1"/>
+      <origin xyz="0 0 0" rpy="0 0 0" />
+      <mass value="10.0" />
+      <inertia ixx="0.1" ixy="0.0" ixz="0.0" iyy="0.1" iyz="0.0" izz="0.1" />
     </inertial>
   </link>
   <!-- create hands -->
-  <xacro:left_hand parent_link="base_link" rail_origin="${lh_start_point}" hand_width="${hand_width}" rail_length="${rail_length}" mesh_dir="${mesh_dir}"/>
-  <xacro:right_hand parent_link="base_link" rail_origin="${rh_start_point}" hand_width="${hand_width}" rail_length="${rail_length}" mesh_dir="${mesh_dir}"/>
+  <xacro:left_hand parent_link="base_link" left_stepper_min="${left_stepper_min}"
+    left_stepper_max="${left_stepper_max}" rail_origin="${lh_start_point}" mesh_dir="${mesh_dir}" />
+  <xacro:right_hand parent_link="base_link" right_stepper_min="${right_stepper_min}"
+    right_stepper_max="${right_stepper_max}" rail_origin="${rh_start_point}" mesh_dir="${mesh_dir}" />
 </robot>

File: src/bothoven_description/urdf/left_hand.xacro (robot description, xacro)
@@ -3,7 +3,5 @@
   <xacro:include filename="$(find bothoven_description)/urdf/finger.xacro" />
   <!-- left hand macro -->
-  <xacro:macro name="left_hand" params="parent_link hand_width rail_origin rail_length mesh_dir">
-    <xacro:property name="half_hand_width" value="${hand_width / 2}" />
-    <xacro:property name="half_rail_length" value="${rail_length / 2}" />
+  <xacro:macro name="left_hand" params="parent_link left_stepper_min left_stepper_max rail_origin mesh_dir">
     <joint name="lh_stepper" type="prismatic">
       <origin xyz="0 ${rail_origin} 0" rpy="0 0 ${pi}" />
@@ -13,6 +11,7 @@
       <!-- limit travel based on the rail length, accounting for hand width, relative to hand
       starting point -->
-      <limit effort="100" velocity="1.0" lower="${-(half_rail_length + rail_origin)}"
-        upper="${half_rail_length - rail_origin - half_hand_width}" />
+      <limit effort="100" velocity="1.0"
+        lower="${left_stepper_min}"
+        upper="${left_stepper_max}" />
     </joint>
     <!-- mount plate link -->

File: src/bothoven_description/urdf/right_hand.xacro (robot description, xacro)
@@ -3,7 +3,5 @@
   <xacro:include filename="$(find bothoven_description)/urdf/finger.xacro" />
   <!-- right hand macro -->
-  <xacro:macro name="right_hand" params="parent_link hand_width rail_origin rail_length mesh_dir">
-    <xacro:property name="half_hand_width" value="${hand_width / 2}" />
-    <xacro:property name="half_rail_length" value="${rail_length / 2}" />
+  <xacro:macro name="right_hand" params="parent_link right_stepper_min right_stepper_max rail_origin mesh_dir">
     <joint name="rh_stepper" type="prismatic">
       <origin xyz="0 ${rail_origin} 0" rpy="0 0 ${pi}" />
@@ -14,6 +12,6 @@
       starting point -->
       <limit effort="100" velocity="1.0"
-        lower="${-(half_rail_length + rail_origin) + half_hand_width}"
-        upper="${half_rail_length - rail_origin}" />
+        lower="${right_stepper_min}"
+        upper="${right_stepper_max}" />
     </joint>
     <!-- mount plate link -->
