Commit message: steppers and solenoids working with gui controller!

File: src/bothoven_description/ros2_control/left_solenoid_joints.xacro (robot description, xacro)
@@ -3,45 +3,45 @@
     <!-- thumb -->
     <joint name="lh_solenoid_1">
-        <command_interface name="position">
+        <command_interface name="position" />
+        <state_interface name="position">
             <param name="min">${solenoid_min}</param>
             <param name="max">${solenoid_max}</param>
-        </command_interface>
-        <state_interface name="position" />
+        </state_interface>
         <param name="solenoid_channel">4</param>
     </joint>
     <!-- index -->
     <joint name="lh_solenoid_2">
-        <command_interface name="position">
+        <command_interface name="position" />
+        <state_interface name="position">
             <param name="min">${solenoid_min}</param>
             <param name="max">${solenoid_max}</param>
-        </command_interface>
-        <state_interface name="position" />
+        </state_interface>
         <param name="solenoid_channel">3</param>
     </joint>
     <!-- middle -->
     <joint name="lh_solenoid_3">
-        <command_interface name="position">
+        <command_interface name="position" />
+        <state_interface name="position">
             <param name="min">${solenoid_min}</param>
             <param name="max">${solenoid_max}</param>
-        </command_interface>
-        <state_interface name="position" />
+        </state_interface>
         <param name="solenoid_channel">2</param>
     </joint>
     <!-- ring -->
     <joint name="lh_solenoid_4">
-        <command_interface name="position">
+        <command_interface name="position" />
+        <state_interface name="position">
             <param name="min">${solenoid_min}</param>
             <param name="max">${solenoid_max}</param>
-        </command_interface>
-        <state_interface name="position" />
+        </state_interface>
         <param name="solenoid_channel">1</param>
     </joint>
     <!-- pinky -->
     <joint name="lh_solenoid_5">
-        <command_interface name="position">
+        <command_interface name="position" />
+        <state_interface name="position">
             <param name="min">${solenoid_min}</param>
             <param name="max">${solenoid_max}</param>
-        </command_interface>
-        <state_interface name="position" />
+        </state_interface>
         <param name="solenoid_channel">0</param>
     </joint>

File: src/bothoven_description/ros2_control/left_stepper_joint.xacro (robot description, xacro)
@@ -2,9 +2,9 @@
 <robot xmlns:xacro="http://www.ros.org/wiki/xacro">
     <joint name="lh_stepper">
-        <command_interface name="position">
+        <command_interface name="velocity" />
+        <state_interface name="position" >
             <param name="min">${left_stepper_min}</param>
             <param name="max">${left_stepper_max}</param>
-        </command_interface>
-        <state_interface name="position" />
+        </state_interface>
     </joint>
 </robot>

File: src/bothoven_description/ros2_control/right_solenoid_joints.xacro (robot description, xacro)
@@ -3,45 +3,45 @@
     <!-- thumb -->
     <joint name="rh_solenoid_1">
-        <command_interface name="position">
+        <command_interface name="position" />
+        <state_interface name="position">
             <param name="min">${solenoid_min}</param>
             <param name="max">${solenoid_max}</param>
-        </command_interface>
-        <state_interface name="position" />
+        </state_interface>
         <param name="solenoid_channel">0</param>
     </joint>
     <!-- index -->
     <joint name="rh_solenoid_2">
-        <command_interface name="position">
+        <command_interface name="position" />
+        <state_interface name="position">
             <param name="min">${solenoid_min}</param>
             <param name="max">${solenoid_max}</param>
-        </command_interface>
-        <state_interface name="position" />
+        </state_interface>
         <param name="solenoid_channel">1</param>
     </joint>
     <!-- middle -->
     <joint name="rh_solenoid_3">
-        <command_interface name="position">
+        <command_interface name="position" />
+        <state_interface name="position">
             <param name="min">${solenoid_min}</param>
             <param name="max">${solenoid_max}</param>
-        </command_interface>
-        <state_interface name="position" />
+        </state_interface>
         <param name="solenoid_channel">2</param>
     </joint>
     <!-- ring -->
     <joint name="rh_solenoid_4">
-        <command_interface name="position">
+        <command_interface name="position" />
+        <state_interface name="position">
             <param name="min">${solenoid_min}</param>
             <param name="max">${solenoid_max}</param>
-        </command_interface>
-        <state_interface name="position" />
+        </state_interface>
         <param name="solenoid_channel">3</param>
     </joint>
     <!-- pinky -->
     <joint name="rh_solenoid_5">
-        <command_interface name="position">
+        <command_interface name="position" />
+        <state_interface name="position">
             <param name="min">${solenoid_min}</param>
             <param name="max">${solenoid_max}</param>
-        </command_interface>
-        <state_interface name="position" />
+        </state_interface>
         <param name="solenoid_channel">4</param>
     </joint>

File: src/bothoven_description/ros2_control/right_stepper_joint.xacro (robot description, xacro)
@@ -2,9 +2,9 @@
 <robot xmlns:xacro="http://www.ros.org/wiki/xacro">
     <joint name="rh_stepper">
-        <command_interface name="position">
+        <command_interface name="velocity" />
+        <state_interface name="position" >
             <param name="min">${right_stepper_min}</param>
             <param name="max">${right_stepper_max}</param>
-        </command_interface>
-        <state_interface name="position" />
+        </state_interface>
     </joint>
 </robot>

File: src/bothoven_description/ros2_control/ros2_control.xacro (robot description, xacro)
@@ -40,4 +40,74 @@
       <xacro:include filename="$(find bothoven_description)/ros2_control/right_stepper_joint.xacro" />
     </ros2_control>
+    <ros2_control name="left_servo_driver" type="system">
+      <xacro:if value="${use_sim}">
+        <hardware>
+          <plugin>gz_ros2_control/GazeboSimSystem</plugin>
+        </hardware>
+      </xacro:if>
+      <xacro:unless value="${use_sim}">
+        <hardware>
+          <plugin>pca9685_hardware_interface/Pca9685SystemHardware</plugin>
+          <param name="i2c_device">/dev/i2c-1</param>
+          <param name="pca_frequency_hz">50</param>
+          <param name="pca_i2c_address">64</param>
+          <param name="min_duty_cycle_ms">0.5</param>
+          <param name="max_duty_cycle_ms">2.5</param>
+          <param name="ads_i2c_address">16</param>          <!-- 0x10 -->
+          <param name="ads_conversion_rate">20</param>          <!-- 20 kSPS -->
+        </hardware>
+      </xacro:unless>
+      <xacro:include filename="$(find bothoven_description)/ros2_control/left_servo_joints.xacro" />
+    </ros2_control>
+    <ros2_control name="right_servo_driver" type="system">
+      <xacro:if value="${use_sim}">
+        <hardware>
+          <plugin>gz_ros2_control/GazeboSimSystem</plugin>
+        </hardware>
+      </xacro:if>
+      <xacro:unless value="${use_sim}">
+        <hardware>
+          <plugin>pca9685_hardware_interface/Pca9685SystemHardware</plugin>
+          <param name="i2c_device">/dev/i2c-1</param>
+          <param name="pca_frequency_hz">50</param>
+          <param name="pca_i2c_address">65</param>
+          <param name="min_duty_cycle_ms">0.5</param>
+          <param name="max_duty_cycle_ms">2.5</param>
+          <param name="ads_i2c_address">18</param>
+          <param name="ads_conversion_rate">20</param>
+        </hardware>
+      </xacro:unless>
+      <xacro:include filename="$(find bothoven_description)/ros2_control/right_servo_joints.xacro" />
+    </ros2_control>
+    <ros2_control name="left_solenoid_driver" type="system">
+      <xacro:if value="${use_sim}">
+        <hardware>
+          <plugin>gz_ros2_control/GazeboSimSystem</plugin>
+        </hardware>
+      </xacro:if>
+      <xacro:unless value="${use_sim}">
+        <hardware>
+          <plugin>mcp23017_hardware_interface/Mcp23017SystemHardware</plugin>
+          <param name="i2c_device">/dev/i2c-1</param>
+          <param name="i2c_address">32</param>
+        </hardware>
+      </xacro:unless>
+      <xacro:include filename="$(find bothoven_description)/ros2_control/left_solenoid_joints.xacro" />
+    </ros2_control>
+    <ros2_control name="right_solenoid_driver" type="system">
+      <xacro:if value="${use_sim}">
+        <hardware>
+          <plugin>gz_ros2_control/GazeboSimSystem</plugin>
+        </hardware>
+      </xacro:if>
+      <xacro:unless value="${use_sim}">
+        <hardware>
+          <plugin>mcp23017_hardware_interface/Mcp23017SystemHardware</plugin>
+          <param name="i2c_device">/dev/i2c-1</param>
+          <param name="i2c_address">33</param>
+        </hardware>
+      </xacro:unless>
+      <xacro:include filename="$(find bothoven_description)/ros2_control/right_solenoid_joints.xacro" />
+    </ros2_control>
   </xacro:macro>
 </robot>

File: src/bothoven_description/urdf/bothoven_core.xacro (robot description, xacro)
@@ -9,5 +9,5 @@
   <xacro:property name="rail_width" value="0.05" />
   <xacro:property name="rail_height" value="0.02" />
-  <xacro:property name="hand_width" value="0.4064" />
+  <xacro:property name="hand_width" value="0.205" />
   <!-- hand origins relative to the rail center -->
   <xacro:property name="lh_start_point" value="-0.3" />
@@ -18,5 +18,6 @@
   <!-- solenoid joint limits -->
   <xacro:property name="solenoid_min" value="0" />
-  <xacro:property name="solenoid_max" value="0.52359877559829881566" />
+  <!-- <xacro:property name="solenoid_max" value="0.52359877559829881566" /> -->
+  <xacro:property name="solenoid_max" value="0.4" />
   <!-- stepper joint limits -->
   <xacro:property name="left_stepper_min" value="${-(rail_length/2 + lh_start_point)}" />
